File: hw/pcb/OrbitESC/input_button.kicad_sch (KiCad schematic)
At the start: 12 parts, among them SW1 Reset, SW2 User, SW3 Boot, SW4 Break

Commit message: Schematic checklist runthrough
Parts:
- SW1, SW2, SW3, SW4: DigiKey (none) -> CKN10502CT-ND
Changed lines of the file:
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@@
+      (effects (font (size 1.27 1.27)) hide)
+    )
+    (property "DigiKey" "CKN10502CT-ND" (id 4) (at 120.65 128.27 0)
       (effects (font (size 1.27 1.27)) hide)
     )
@@
       (effects (font (size 1.27 1.27)) hide)
     )
+    (property "DigiKey" "CKN10502CT-ND" (id 4) (at 146.05 66.04 0)
+      (effects (font (size 1.27 1.27)) hide)
+    )
     (pin "1")
     (pin "2")
@@
       (effects (font (size 1.27 1.27)) hide)
     )
+    (property "DigiKey" "CKN10502CT-ND" (id 4) (at 146.05 128.27 0)
+      (effects (font (size 1.27 1.27)) hide)
+    )
     (pin "1")
     (pin "2")
@@
       (effects (font (size 1.27 1.27)) hide)
     )
+    (property "DigiKey" "CKN10502CT-ND" (id 4) (at 120.65 77.47 0)
+      (effects (font (size 1.27 1.27)) hide)
+    )

Commit message: Start rework of processor selection after realizing I can't afford manufacturing...
Parts:
- removed C31, C32: 100nF, Capacitor_SMD:C_0402_1005Metric, symbol Device:C
- removed R54, R56, R57: 10k, Resistor_SMD:R_0402_1005Metric, symbol Device:R_US
- removed SW2: User, Button_Switch_SMD:SW_SPST_PTS810, symbol Switch:SW_Push
- removed SW4: Break, Button_Switch_SMD:SW_SPST_PTS810, symbol Switch:SW_Push
