File: hw/pcb/OrbitESC/status_leds.kicad_sch (KiCad schematic)
At the start: 18 parts, among them U12 74HC595

Commit message: Sync PCB updates
Parts:
- R7: value 1.5k -> 470; JLCPCB C25867 -> C25117
- R87, R88, R90: value 200 -> 470; JLCPCB C25087 -> C25117
Other:
- note removed: "Match the LED MCD properties to be similar to the green ones"
Changed lines of the file:
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@@
     (stroke (width 0) (type default) (color 0 0 0 0))
-  )
-  (text "Match the LED MCD properties to be similar to the green ones"
-    (at 146.685 63.5 0)
-    (effects (font (size 1.27 1.27)) (justify left bottom))
   )
   (label "FAULT" (at 137.16 66.04 0)
@@
       (effects (font (size 1.27 1.27)) (justify left))
     )
-    (property "Value" "200" (id 1) (at 161.29 106.6799 0)
+    (property "Value" "470" (id 1) (at 161.29 106.6799 0)
       (effects (font (size 1.27 1.27)) (justify left))
     )
@@
       (effects (font (size 1.27 1.27)) hide)
     )
-    (property "JLCPCB" "C25087" (id 4) (at 158.75 105.41 0)
+    (property "JLCPCB" "C25117" (id 4) (at 158.75 105.41 0)
       (effects (font (size 1.27 1.27)) hide)
     )
@@
       (effects (font (size 1.27 1.27)) (justify left))
     )
-    (property "Value" "200" (id 1) (at 152.4 106.6799 0)
+    (property "Value" "470" (id 1) (at 152.4 106.6799 0)
       (effects (font (size 1.27 1.27)) (justify left))
     )
@@
       (effects (font (size 1.27 1.27)) hide)
     )
-    (property "JLCPCB" "C25087" (id 4) (at 149.86 105.41 0)
+    (property "JLCPCB" "C25117" (id 4) (at 149.86 105.41 0)
       (effects (font (size 1.27 1.27)) hide)
     )
@@
       (effects (font (size 1.27 1.27)) (justify left))
     )
-    (property "Value" "200" (id 1) (at 170.18 106.6799 0)
+    (property "Value" "470" (id 1) (at 170.18 106.6799 0)
       (effects (font (size 1.27 1.27)) (justify left))
     )
@@
       (effects (font (size 1.27 1.27)) hide)
     )
-    (property "JLCPCB" "C25087" (id 4) (at 167.64 105.41 0)
+    (property "JLCPCB" "C25117" (id 4) (at 167.64 105.41 0)
       (effects (font (size 1.27 1.27)) hide)
     )
@@
       (effects (font (size 1.27 1.27)) (justify left))
     )
-    (property "Value" "1.5k" (id 1) (at 143.51 106.6799 0)
+    (property "Value" "470" (id 1) (at 143.51 106.6799 0)
       (effects (font (size 1.27 1.27)) (justify left))
     )
@@
       (effects (font (size 1.27 1.27)) hide)
     )
-    (property "JLCPCB" "C25867" (id 4) (at 140.97 105.41 0)
-      (effects (font (size 1.27 1.27)) hide)
-    )
+    (property "JLCPCB" "C25117" (id 4) (at 140.97 105.41 0)
+      (effects (font (size 1.27 1.27)) hide)
+    )

Commit message: Finalize V2 PCB
Parts:
- C32: JLCPCB C307331 -> (none); LCSC (none) -> C307331
- D15, D18: JLCPCB C72043 -> (none); LCSC (none) -> C72043
- D16, D17, D19: JLCPCB C72041 -> (none); LCSC (none) -> C72041
- D20: JLCPCB C2286 -> (none); LCSC (none) -> C2286
- D5: JLCPCB C72038 -> (none); LCSC (none) -> C72038
- R19, R29, R86, R89: JLCPCB C25744 -> (none); LCSC (none) -> C25744
- R7, R87, R88, R90: JLCPCB C25117 -> (none); LCSC (none) -> C25117
- R91: JLCPCB C25867 -> (none); LCSC (none) -> C25867
- U12: value 74HC595 -> MC74HC595ADTR2G; footprint Package_SO:SOIC-16_3.9x9.9mm_P1.27mm -> Package_SO:TSSOP-16_4.4x5mm_P0.65mm; JLCPCB C5947 -> (none); LCSC (none) -> C100027
Connections:
- net CAN1_ACTV: now also U12.3 (QD); no longer U12.6 (QG)
- net STATUS_0: now also U12.4 (QE); no longer U12.3 (QD)
- net STATUS_1: now also U12.5 (QF); no longer U12.4 (QE)
- net STATUS_2: now also U12.6 (QG); no longer U12.5 (QF)
Other:
- moved on the sheet: D16, D17, D19, D5, R7, R87, R88, R90
