File: hw/pcb/OrbitESC/output_stage.kicad_sch (KiCad schematic)
At the start: 24 parts, among them J3 TermA, J4 TermB, J5 TermC, Q1 MCAC80N10Y, Q2 MCAC80N10Y, Q3 MCAC80N10Y, Q4 MCAC80N10Y, Q5 MCAC80N10Y, Q6 MCAC80N10Y

Commit message: Improve power section layout
Parts:
- C2, C5, C8: footprint Capacitor_SMD:C_0603_1608Metric -> Capacitor_SMD:C_0402_1005Metric; JLCPCB C1588 -> C1523
Changed lines of the file:
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@@
       (effects (font (size 1.27 1.27)) (justify left))
     )
-    (property "Footprint" "Capacitor_SMD:C_0603_1608Metric" (id 2) (at 158.4452 118.11 0)
+    (property "Footprint" "Capacitor_SMD:C_0402_1005Metric" (id 2) (at 158.4452 118.11 0)
       (effects (font (size 1.27 1.27)) hide)
     )
@@
       (effects (font (size 1.27 1.27)) hide)
     )
-    (property "JLCPCB" "C1588" (id 4) (at 157.48 114.3 0)
+    (property "JLCPCB" "C1523" (id 4) (at 157.48 114.3 0)
       (effects (font (size 1.27 1.27)) hide)
     )
@@
       (effects (font (size 1.27 1.27)) (justify left))
     )
-    (property "Footprint" "Capacitor_SMD:C_0603_1608Metric" (id 2) (at 246.0752 118.11 0)
+    (property "Footprint" "Capacitor_SMD:C_0402_1005Metric" (id 2) (at 246.0752 118.11 0)
       (effects (font (size 1.27 1.27)) hide)
     )
@@
       (effects (font (size 1.27 1.27)) hide)
     )
-    (property "JLCPCB" "C1588" (id 4) (at 245.11 114.3 0)
+    (property "JLCPCB" "C1523" (id 4) (at 245.11 114.3 0)
       (effects (font (size 1.27 1.27)) hide)
     )
@@
       (effects (font (size 1.27 1.27)) (justify left))
     )
-    (property "Footprint" "Capacitor_SMD:C_0603_1608Metric" (id 2) (at 70.8152 118.11 0)
+    (property "Footprint" "Capacitor_SMD:C_0402_1005Metric" (id 2) (at 70.8152 118.11 0)
       (effects (font (size 1.27 1.27)) hide)
     )
@@
       (effects (font (size 1.27 1.27)) hide)
     )
-    (property "JLCPCB" "C1588" (id 4) (at 69.85 114.3 0)
+    (property "JLCPCB" "C1523" (id 4) (at 69.85 114.3 0)
       (effects (font (size 1.27 1.27)) hide)
     )

Commit message: Sync today's work
Parts:
- added C37: 2.2uF, Capacitor_SMD:C_0805_2012Metric, symbol Device:C
Connections:
- net GND: now also C37.2
- net VDC: now also C37.1
Changed lines of the file:
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@@
     (pin "2")
+  )
+  (symbol (lib_id "power:VDC") (at 113.03 46.355 0) (unit 1)
+    (in_bom yes) (on_board yes) (fields_autoplaced)
+    (property "Reference" "#PWR035" (id 0) (at 113.03 48.895 0)
+      (effects (font (size 1.27 1.27)) hide)
+    )
+    (property "Value" "VDC" (id 1) (at 113.03 41.275 0))
+    (property "Footprint" "" (id 2) (at 113.03 46.355 0)
+      (effects (font (size 1.27 1.27)) hide)
+    )
+    (property "Datasheet" "" (id 3) (at 113.03 46.355 0)
+      (effects (font (size 1.27 1.27)) hide)
+    )
+    (pin "1")
   )
   (symbol (lib_id "Project Mosfets:MCAC80N10Y") (at 252.73 71.12 0) (unit 1)
@@
     (pin "2")
   )
+  (symbol (lib_id "power:GND") (at 113.03 53.975 0) (unit 1)
+    (in_bom yes) (on_board yes) (fields_autoplaced)
+    (property "Reference" "#PWR086" (id 0) (at 113.03 60.325 0)
+      (effects (font (size 1.27 1.27)) hide)
+    )
+    (property "Value" "GND" (id 1) (at 113.03 59.055 0))
+    (property "Footprint" "" (id 2) (at 113.03 53.975 0)
+      (effects (font (size 1.27 1.27)) hide)
+    )
+    (property "Datasheet" "" (id 3) (at 113.03 53.975 0)
+      (effects (font (size 1.27 1.27)) hide)
+    )
+    (pin "1")
+  )
   (symbol (lib_id "Device:R_US") (at 151.13 97.79 90) (unit 1)
     (in_bom yes) (on_board yes) (fields_autoplaced)
@@
       (effects (font (size 1.27 1.27)) hide)
     )
+    (pin "1")
+    (pin "2")
+  )
+  (symbol (lib_id "Device:C") (at 113.03 50.165 0) (unit 1)
+    (in_bom yes) (on_board yes) (fields_autoplaced)
+    (property "Reference" "C37" (id 0) (at 116.84 48.8949 0)
+      (effects (font (size 1.27 1.27)) (justify left))
+    )
+    (property "Value" "2.2uF" (id 1) (at 116.84 51.4349 0)
+      (effects (font (size 1.27 1.27)) (justify left))
+    )
+    (property "Footprint" "Capacitor_SMD:C_0805_2012Metric" (id 2) (at 113.9952 53.975 0)
+      (effects (font (size 1.27 1.27)) hide)
+    )
+    (property "Datasheet" "~" (id 3) (at 113.03 50.165 0)
+      (effects (font (size 1.27 1.27)) hide)
+    )
+    (property "JLCPCB" "C49217" (id 4) (at 113.03 50.165 0)
+      (effects (font (size 1.27 1.27)) hide)
+    )
