File: hw/pcb/OrbitESC/output_stage.kicad_sch (KiCad schematic)
At the start: 25 parts, among them J3 TermA, J4 TermB, J5 TermC, Q1 MCAC80N10Y, Q2 MCAC80N10Y, Q3 MCAC80N10Y, Q4 MCAC80N10Y, Q5 MCAC80N10Y, Q6 MCAC80N10Y

Commit message: Finalize V2 PCB
Parts:
- C2, C5, C8: JLCPCB C1523 -> (none); LCSC (none) -> C1523
- C3, C37, C6, C9: JLCPCB C49217 -> (none); LCSC (none) -> C49217
- Q1, Q2, Q3, Q4, Q5, Q6: value MCAC80N10Y -> MCAC100N08YA-TP; DigiKey 353-MCAC80N10Y-TPCT-ND -> 353-MCAC100N08YA-TPCT-ND
- R10, R14, R16, R2, R4, R8: JLCPCB C25086 -> (none); LCSC (none) -> C25086
Changed lines of the file:
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@@
       (effects (font (size 1.27 1.27)) hide)
     )
-    (property "JLCPCB" "C49217" (id 4) (at 186.69 68.58 0)
+    (property "JLCPCB" "" (id 4) (at 186.69 68.58 0)
+      (effects (font (size 1.27 1.27)) hide)
+    )
+    (property "LCSC" "C49217" (id 5) (at 186.69 68.58 0)
       (effects (font (size 1.27 1.27)) hide)
     )
@@
       (effects (font (size 1.27 1.27)) (justify left))
     )
-    (property "Value" "MCAC80N10Y" (id 1) (at 171.45 99.0599 0)
+    (property "Value" "MCAC100N08YA-TP" (id 1) (at 171.45 99.0599 0)
       (effects (font (size 1.27 1.27)) (justify left))
     )
@@
       (effects (font (size 1.27 1.27)) hide)
     )
-    (property "Datasheet" "https://www.mccsemi.com/pdf/Products/MCAC80N10Y(DFN5060).pdf" (id 3) (at 165.1 97.79 0)
-      (effects (font (size 1.27 1.27)) hide)
-    )
-    (property "DigiKey" "353-MCAC80N10Y-TPCT-ND" (id 4) (at 165.1 97.79 0)
+    (property "Datasheet" "https://www.mccsemi.com/pdf/Products/MCAC100N08YA(DFN5060).pdf" (id 3) (at 165.1 97.79 0)
+      (effects (font (size 1.27 1.27)) hide)
+    )
+    (property "DigiKey" "353-MCAC100N08YA-TPCT-ND" (id 4) (at 165.1 97.79 0)
       (effects (font (size 1.27 1.27)) hide)
     )
@@
       (effects (font (size 1.27 1.27)) (justify left))
     )
-    (property "Value" "MCAC80N10Y" (id 1) (at 171.45 72.3899 0)
+    (property "Value" "MCAC100N08YA-TP" (id 1) (at 171.45 72.3899 0)
       (effects (font (size 1.27 1.27)) (justify left))
     )
@@
       (effects (font (size 1.27 1.27)) hide)
     )
-    (property "Datasheet" "https://www.mccsemi.com/pdf/Products/MCAC80N10Y(DFN5060).pdf" (id 3) (at 165.1 71.12 0)
-      (effects (font (size 1.27 1.27)) hide)
-    )
-    (property "DigiKey" "353-MCAC80N10Y-TPCT-ND" (id 4) (at 165.1 71.12 0)
+    (property "Datasheet" "https://www.mccsemi.com/pdf/Products/MCAC100N08YA(DFN5060).pdf" (id 3) (at 165.1 71.12 0)
+      (effects (font (size 1.27 1.27)) hide)
+    )
+    (property "DigiKey" "353-MCAC100N08YA-TPCT-ND" (id 4) (at 165.1 71.12 0)
       (effects (font (size 1.27 1.27)) hide)
     )
@@
       (effects (font (size 1.27 1.27)) hide)
     )
-    (property "JLCPCB" "C25086" (id 4) (at 63.5 71.12 90)
+    (property "JLCPCB" "" (id 4) (at 63.5 71.12 90)
+      (effects (font (size 1.27 1.27)) hide)
+    )
+    (property "LCSC" "C25086" (id 5) (at 63.5 71.12 0)
       (effects (font (size 1.27 1.27)) hide)
     )
@@
       (effects (font (size 1.27 1.27)) hide)
     )
-    (property "JLCPCB" "C49217" (id 4) (at 274.32 68.58 0)
+    (property "JLCPCB" "" (id 4) (at 274.32 68.58 0)
+      (effects (font (size 1.27 1.27)) hide)
+    )
+    (property "LCSC" "C49217" (id 5) (at 274.32 68.58 0)
       (effects (font (size 1.27 1.27)) hide)
     )
@@
       (effects (font (size 1.27 1.27)) (justify left))
     )
-    (property "Value" "MCAC80N10Y" (id 1) (at 259.08 72.3899 0)
+    (property "Value" "MCAC100N08YA-TP" (id 1) (at 259.08 72.3899 0)
       (effects (font (size 1.27 1.27)) (justify left))
     )
@@
       (effects (font (size 1.27 1.27)) hide)
     )
-    (property "Datasheet" "https://www.mccsemi.com/pdf/Products/MCAC80N10Y(DFN5060).pdf" (id 3) (at 252.73 71.12 0)
-      (effects (font (size 1.27 1.27)) hide)
-    )
-    (property "DigiKey" "353-MCAC80N10Y-TPCT-ND" (id 4) (at 252.73 71.12 0)
+    (property "Datasheet" "https://www.mccsemi.com/pdf/Products/MCAC100N08YA(DFN5060).pdf" (id 3) (at 252.73 71.12 0)
+      (effects (font (size 1.27 1.27)) hide)
+    )
+    (property "DigiKey" "353-MCAC100N08YA-TPCT-ND" (id 4) (at 252.73 71.12 0)
       (effects (font (size 1.27 1.27)) hide)
     )
@@
       (effects (font (size 1.27 1.27)) (justify left))
     )
-    (property "Value" "MCAC80N10Y" (id 1) (at 83.82 72.3899 0)
+    (property "Value" "MCAC100N08YA-TP" (id 1) (at 83.82 72.3899 0)
       (effects (font (size 1.27 1.27)) (justify left))
     )
@@
       (effects (font (size 1.27 1.27)) hide)
     )
-    (property "Datasheet" "https://www.mccsemi.com/pdf/Products/MCAC80N10Y(DFN5060).pdf" (id 3) (at 77.47 71.12 0)
-      (effects (font (size 1.27 1.27)) hide)
-    )
-    (property "DigiKey" "353-MCAC80N10Y-TPCT-ND" (id 4) (at 77.47 71.12 0)
+    (property "Datasheet" "https://www.mccsemi.com/pdf/Products/MCAC100N08YA(DFN5060).pdf" (id 3) (at 77.47 71.12 0)
+      (effects (font (size 1.27 1.27)) hide)
+    )
+    (property "DigiKey" "353-MCAC100N08YA-TPCT-ND" (id 4) (at 77.47 71.12 0)
       (effects (font (size 1.27 1.27)) hide)
     )
@@
       (effects (font (size 1.27 1.27)) (justify left))
     )
-    (property "Value" "MCAC80N10Y" (id 1) (at 259.08 99.0599 0)
+    (property "Value" "MCAC100N08YA-TP" (id 1) (at 259.08 99.0599 0)
       (effects (font (size 1.27 1.27)) (justify left))
     )
@@
       (effects (font (size 1.27 1.27)) hide)
     )
-    (property "Datasheet" "https://www.mccsemi.com/pdf/Products/MCAC80N10Y(DFN5060).pdf" (id 3) (at 252.73 97.79 0)
-      (effects (font (size 1.27 1.27)) hide)
-    )
-    (property "DigiKey" "353-MCAC80N10Y-TPCT-ND" (id 4) (at 252.73 97.79 0)
+    (property "Datasheet" "https://www.mccsemi.com/pdf/Products/MCAC100N08YA(DFN5060).pdf" (id 3) (at 252.73 97.79 0)
+      (effects (font (size 1.27 1.27)) hide)
+    )
+    (property "DigiKey" "353-MCAC100N08YA-TPCT-ND" (id 4) (at 252.73 97.79 0)
       (effects (font (size 1.27 1.27)) hide)
     )
@@
       (effects (font (size 1.27 1.27)) hide)
     )
-    (property "JLCPCB" "C1523" (id 4) (at 157.48 114.3 0)
+    (property "JLCPCB" "" (id 4) (at 157.48 114.3 0)
+      (effects (font (size 1.27 1.27)) hide)
+    )
+    (property "LCSC" "C1523" (id 5) (at 157.48 114.3 0)
       (effects (font (size 1.27 1.27)) hide)
     )
@@
       (effects (font (size 1.27 1.27)) hide)
     )
-    (property "JLCPCB" "C25086" (id 4) (at 238.76 97.79 90)
+    (property "JLCPCB" "" (id 4) (at 238.76 97.79 90)
+      (effects (font (size 1.27 1.27)) hide)
+    )
+    (property "LCSC" "C25086" (id 5) (at 238.76 97.79 0)
       (effects (font (size 1.27 1.27)) hide)
     )
@@
       (effects (font (size 1.27 1.27)) hide)
     )
-    (property "JLCPCB" "C1523" (id 4) (at 245.11 114.3 0)
+    (property "JLCPCB" "" (id 4) (at 245.11 114.3 0)
+      (effects (font (size 1.27 1.27)) hide)
+    )
+    (property "LCSC" "C1523" (id 5) (at 245.11 114.3 0)
       (effects (font (size 1.27 1.27)) hide)
     )
@@
       (effects (font (size 1.27 1.27)) hide)
     )
-    (property "JLCPCB" "C49217" (id 4) (at 99.06 68.58 0)
+    (property "JLCPCB" "" (id 4) (at 99.06 68.58 0)
+      (effects (font (size 1.27 1.27)) hide)
+    )
+    (property "LCSC" "C49217" (id 5) (at 99.06 68.58 0)
       (effects (font (size 1.27 1.27)) hide)
     )
@@
       (effects (font (size 1.27 1.27)) (justify left))
     )
-    (property "Value" "MCAC80N10Y" (id 1) (at 83.82 99.0599 0)
+    (property "Value" "MCAC100N08YA-TP" (id 1) (at 83.82 99.0599 0)
       (effects (font (size 1.27 1.27)) (justify left))
     )
@@
       (effects (font (size 1.27 1.27)) hide)
     )
-    (property "Datasheet" "https://www.mccsemi.com/pdf/Products/MCAC80N10Y(DFN5060).pdf" (id 3) (at 77.47 97.79 0)
-      (effects (font (size 1.27 1.27)) hide)
-    )
-    (property "DigiKey" "353-MCAC80N10Y-TPCT-ND" (id 4) (at 77.47 97.79 0)
+    (property "Datasheet" "https://www.mccsemi.com/pdf/Products/MCAC100N08YA(DFN5060).pdf" (id 3) (at 77.47 97.79 0)
+      (effects (font (size 1.27 1.27)) hide)
+    )
+    (property "DigiKey" "353-MCAC100N08YA-TPCT-ND" (id 4) (at 77.47 97.79 0)
       (effects (font (size 1.27 1.27)) hide)
     )
@@
       (effects (font (size 1.27 1.27)) hide)
     )
-    (property "JLCPCB" "C25086" (id 4) (at 151.13 71.12 90)
+    (property "JLCPCB" "" (id 4) (at 151.13 71.12 90)
+      (effects (font (size 1.27 1.27)) hide)
+    )
+    (property "LCSC" "C25086" (id 5) (at 151.13 71.12 0)
       (effects (font (size 1.27 1.27)) hide)
     )
@@
       (effects (font (size 1.27 1.27)) hide)
     )
-    (property "JLCPCB" "C25086" (id 4) (at 151.13 97.79 90)
+    (property "JLCPCB" "" (id 4) (at 151.13 97.79 90)
+      (effects (font (size 1.27 1.27)) hide)
+    )
+    (property "LCSC" "C25086" (id 5) (at 151.13 97.79 0)
       (effects (font (size 1.27 1.27)) hide)
     )
@@
       (effects (font (size 1.27 1.27)) hide)
     )
-    (property "JLCPCB" "C1523" (id 4) (at 69.85 114.3 0)
+    (property "JLCPCB" "" (id 4) (at 69.85 114.3 0)
+      (effects (font (size 1.27 1.27)) hide)
+    )
+    (property "LCSC" "C1523" (id 5) (at 69.85 114.3 0)
       (effects (font (size 1.27 1.27)) hide)
     )
@@
       (effects (font (size 1.27 1.27)) hide)
     )
-    (property "JLCPCB" "C25086" (id 4) (at 238.76 71.12 90)
+    (property "JLCPCB" "" (id 4) (at 238.76 71.12 90)
+      (effects (font (size 1.27 1.27)) hide)
+    )
+    (property "LCSC" "C25086" (id 5) (at 238.76 71.12 0)
       (effects (font (size 1.27 1.27)) hide)
     )
@@
       (effects (font (size 1.27 1.27)) hide)
     )
-    (property "JLCPCB" "C49217" (id 4) (at 113.03 50.165 0)
+    (property "JLCPCB" "" (id 4) (at 113.03 50.165 0)
+      (effects (font (size 1.27 1.27)) hide)
+    )
+    (property "LCSC" "C49217" (id 5) (at 113.03 50.165 0)
       (effects (font (size 1.27 1.27)) hide)
     )
@@
       (effects (font (size 1.27 1.27)) hide)
     )
-    (property "JLCPCB" "C25086" (id 4) (at 63.5 97.79 90)
-      (effects (font (size 1.27 1.27)) hide)
-    )
+    (property "JLCPCB" "" (id 4) (at 63.5 97.79 90)
+      (effects (font (size 1.27 1.27)) hide)
+    )
+    (property "LCSC" "C25086" (id 5) (at 63.5 97.79 0)
+      (effects (font (size 1.27 1.27)) hide)
+    )
