File: hw/pcb/OrbitESC/USB2Serial.kicad_sch (KiCad schematic)
At the start: 12 parts, among them J1 USB_C_Receptacle_USB2.0, U10 CP2104

Commit message: Schematic corrections
Parts:
- removed D6, D7: Yellow LED, Diode_SMD:D_0603_1608Metric, symbol Device:LED
- removed R19, R20: 1.5k, Resistor_SMD:R_0402_1005Metric, symbol Device:R_US
Connections:
- no-connect marks 13 -> 15
Changed lines of the file:
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@@
   (junction (at 140.335 72.39) (diameter 0) (color 0 0 0 0)
-  )
-  (junction (at 196.215 99.695) (diameter 0) (color 0 0 0 0)
   )
   (junction (at 142.875 115.57) (diameter 0) (color 0 0 0 0)
@@
   (no_connect (at 102.87 106.68))
   (no_connect (at 102.87 104.14))
+  (no_connect (at 170.18 102.87))
   (no_connect (at 170.18 107.95))
   (no_connect (at 170.18 90.17))
@@
   (no_connect (at 170.18 77.47))
   (no_connect (at 170.18 95.25))
+  (no_connect (at 170.18 105.41))
   (wire (pts (xy 160.02 64.135) (xy 160.02 67.31))
     (stroke (width 0) (type default) (color 0 0 0 0))
@@
     (stroke (width 0) (type default) (color 0 0 0 0))
   )
-  (wire (pts (xy 196.215 99.695) (xy 196.215 106.68))
-    (stroke (width 0) (type default) (color 0 0 0 0))
-  )
   (wire (pts (xy 104.14 91.44) (xy 102.87 91.44))
     (stroke (width 0) (type default) (color 0 0 0 0))
   )
-  (wire (pts (xy 170.18 105.41) (xy 173.355 105.41))
-    (stroke (width 0) (type default) (color 0 0 0 0))
-  )
   (wire (pts (xy 142.875 115.57) (xy 142.875 116.205))
     (stroke (width 0) (type default) (color 0 0 0 0))
@@
     (stroke (width 0) (type default) (color 0 0 0 0))
   )
-  (wire (pts (xy 173.355 106.68) (xy 177.165 106.68))
-    (stroke (width 0) (type default) (color 0 0 0 0))
-  )
   (wire (pts (xy 140.335 72.39) (xy 144.78 72.39))
     (stroke (width 0) (type default) (color 0 0 0 0))
@@
     (stroke (width 0) (type default) (color 0 0 0 0))
   )
-  (wire (pts (xy 196.215 97.79) (xy 196.215 99.695))
-    (stroke (width 0) (type default) (color 0 0 0 0))
-  )
-  (wire (pts (xy 173.355 99.695) (xy 177.165 99.695))
-    (stroke (width 0) (type default) (color 0 0 0 0))
-  )
-  (wire (pts (xy 196.215 99.695) (xy 192.405 99.695))
-    (stroke (width 0) (type default) (color 0 0 0 0))
-  )
   (wire (pts (xy 154.94 64.135) (xy 154.94 67.31))
     (stroke (width 0) (type default) (color 0 0 0 0))
   )
-  (wire (pts (xy 196.215 106.68) (xy 192.405 106.68))
-    (stroke (width 0) (type default) (color 0 0 0 0))
-  )
-  (wire (pts (xy 173.355 105.41) (xy 173.355 106.68))
-    (stroke (width 0) (type default) (color 0 0 0 0))
-  )
-  (wire (pts (xy 173.355 102.87) (xy 173.355 99.695))
-    (stroke (width 0) (type default) (color 0 0 0 0))
-  )
   (wire (pts (xy 110.49 81.28) (xy 111.76 81.28))
     (stroke (width 0) (type default) (color 0 0 0 0))
@@
   )
   (wire (pts (xy 137.795 116.205) (xy 137.795 115.57))
-    (stroke (width 0) (type default) (color 0 0 0 0))
-  )
-  (wire (pts (xy 170.18 102.87) (xy 173.355 102.87))
     (stroke (width 0) (type default) (color 0 0 0 0))
   )
@@
     (pin "1")
     (pin "2")
-  )
-  (symbol (lib_id "power:+3.3V") (at 196.215 97.79 0) (unit 1)
-    (in_bom yes) (on_board yes) (fields_autoplaced)
-    (property "Reference" "#PWR054" (id 0) (at 196.215 101.6 0)
-      (effects (font (size 1.27 1.27)) hide)
-    )
-    (property "Value" "+3.3V" (id 1) (at 196.215 92.71 0))
-    (property "Footprint" "" (id 2) (at 196.215 97.79 0)
-      (effects (font (size 1.27 1.27)) hide)
-    )
-    (property "Datasheet" "" (id 3) (at 196.215 97.79 0)
-      (effects (font (size 1.27 1.27)) hide)
-    )
-    (pin "1")
   )
   (symbol (lib_id "power:GNDD") (at 137.795 123.825 0) (unit 1)
@@
     (pin "B9")
     (pin "S1")
-  )
-  (symbol (lib_id "Device:LED") (at 180.975 99.695 0) (unit 1)
-    (in_bom yes) (on_board yes)
-    (property "Reference" "D6" (id 0) (at 185.42 100.965 0)
-      (effects (font (size 1.27 1.27)) (justify right))
-    )
-    (property "Value" "Yellow LED" (id 1) (at 186.69 97.155 0)
-      (effects (font (size 1.27 1.27)) (justify right))
-    )
-    (property "Footprint" "Diode_SMD:D_0603_1608Metric" (id 2) (at 180.975 99.695 0)
-      (effects (font (size 1.27 1.27)) hide)
-    )
-    (property "Datasheet" "~" (id 3) (at 180.975 99.695 0)
-      (effects (font (size 1.27 1.27)) hide)
-    )
-    (property "JLCPCB" "C72038" (id 4) (at 180.975 99.695 90)
-      (effects (font (size 1.27 1.27)) hide)
-    )
-    (pin "1")
-    (pin "2")
   )
   (symbol (lib_id "Interface_USB:CP2104") (at 157.48 95.25 0) (unit 1)
@@
     (pin "2")
   )
-  (symbol (lib_id "Device:LED") (at 180.975 106.68 0) (unit 1)
-    (in_bom yes) (on_board yes)
-    (property "Reference" "D7" (id 0) (at 185.42 107.95 0)
-      (effects (font (size 1.27 1.27)) (justify right))
-    )
-    (property "Value" "Yellow LED" (id 1) (at 186.69 104.14 0)
-      (effects (font (size 1.27 1.27)) (justify right))
-    )
-    (property "Footprint" "Diode_SMD:D_0603_1608Metric" (id 2) (at 180.975 106.68 0)
-      (effects (font (size 1.27 1.27)) hide)
-    )
-    (property "Datasheet" "~" (id 3) (at 180.975 106.68 0)
-      (effects (font (size 1.27 1.27)) hide)
-    )
-    (property "JLCPCB" "C72038" (id 4) (at 180.975 106.68 90)
-      (effects (font (size 1.27 1.27)) hide)
-    )
-    (pin "1")
-    (pin "2")
-  )
   (symbol (lib_id "power:+3.3V") (at 160.02 64.135 0) (unit 1)
     (in_bom yes) (on_board yes) (fields_autoplaced)
@@
       (effects (font (size 1.27 1.27)) hide)
     )
-    (pin "1")
-    (pin "2")
-  )
-  (symbol (lib_id "Device:R_US") (at 188.595 106.68 270) (unit 1)
-    (in_bom yes) (on_board yes)
-    (property "Reference" "R20" (id 0) (at 187.96 104.14 90)
-      (effects (font (size 1.27 1.27)) (justify left))
-    )
-    (property "Value" "1.5k" (id 1) (at 187.3251 109.22 90)
-      (effects (font (size 1.27 1.27)) (justify left))
-    )
-    (property "Footprint" "Resistor_SMD:R_0402_1005Metric" (id 2) (at 188.341 107.696 90)
-      (effects (font (size 1.27 1.27)) hide)
-    )
-    (property "Datasheet" "~" (id 3) (at 188.595 106.68 0)
-      (effects (font (size 1.27 1.27)) hide)
-    )
-    (property "JLCPCB" "C25867" (id 4) (at 188.595 106.68 0)
-      (effects (font (size 1.27 1.27)) hide)
-    )
-    (pin "1")
-    (pin "2")
-  )
-  (symbol (lib_id "Device:R_US") (at 188.595 99.695 270) (unit 1)
-    (in_bom yes) (on_board yes)
-    (property "Reference" "R19" (id 0) (at 187.96 97.155 90)
-      (effects (font (size 1.27 1.27)) (justify left))
-    )
-    (property "Value" "1.5k" (id 1) (at 187.3251 102.235 90)
-      (effects (font (size 1.27 1.27)) (justify left))
-    )
-    (property "Footprint" "Resistor_SMD:R_0402_1005Metric" (id 2) (at 188.341 100.711 90)
-      (effects (font (size 1.27 1.27)) hide)
-    )
-    (property "Datasheet" "~" (id 3) (at 188.595 99.695 0)
-      (effects (font (size 1.27 1.27)) hide)
-    )
-    (property "JLCPCB" "C25867" (id 4) (at 188.595 99.695 0)
-      (effects (font (size 1.27 1.27)) hide)
-    )

Commit message: Finalize V2 PCB
Parts:
- removed C10: 2.2uF, Capacitor_SMD:C_0805_2012Metric, symbol Device:C
- C4, C7: value 2.2uF -> 47uF; JLCPCB C49217 -> (none); LCSC (none) -> C16780
- R13, R9: LCSC (none) -> C25905
- R15: JLCPCB C25744 -> (none); LCSC (none) -> C25744
Connections:
- net GNDD: now also C4.2, C7.2; no longer C4.1, C7.1
- net VBUS: now also C4.1; no longer C4.2
- net at U10.16 (VPP): now also C7.1; no longer C7.2
Changed lines of the file:
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@@
   (junction (at 140.335 72.39) (diameter 0) (color 0 0 0 0)
-  )
-  (junction (at 142.875 115.57) (diameter 0) (color 0 0 0 0)
   )
   (no_connect (at 157.48 67.31))
@@
     (stroke (width 0) (type default) (color 0 0 0 0))
   )
-  (wire (pts (xy 142.875 115.57) (xy 144.78 115.57))
+  (wire (pts (xy 138.43 115.57) (xy 138.43 116.205))
     (stroke (width 0) (type default) (color 0 0 0 0))
   )
@@
     (stroke (width 0) (type default) (color 0 0 0 0))
   )
-  (wire (pts (xy 142.875 115.57) (xy 142.875 116.205))
-    (stroke (width 0) (type default) (color 0 0 0 0))
-  )
   (wire (pts (xy 102.87 96.52) (xy 104.14 96.52))
     (stroke (width 0) (type default) (color 0 0 0 0))
@@
     (stroke (width 0) (type default) (color 0 0 0 0))
   )
+  (wire (pts (xy 144.78 115.57) (xy 138.43 115.57))
+    (stroke (width 0) (type default) (color 0 0 0 0))
+  )
   (wire (pts (xy 154.94 64.135) (xy 154.94 67.31))
     (stroke (width 0) (type default) (color 0 0 0 0))
   )
   (wire (pts (xy 110.49 81.28) (xy 111.76 81.28))
-    (stroke (width 0) (type default) (color 0 0 0 0))
-  )
-  (wire (pts (xy 137.795 115.57) (xy 142.875 115.57))
-    (stroke (width 0) (type default) (color 0 0 0 0))
-  )
-  (wire (pts (xy 137.795 116.205) (xy 137.795 115.57))
     (stroke (width 0) (type default) (color 0 0 0 0))
   )
@@
     (pin "1")
   )
-  (symbol (lib_id "Device:C") (at 137.795 120.015 0) (mirror x) (unit 1)
-    (in_bom yes) (on_board yes) (fields_autoplaced)
-    (property "Reference" "C7" (id 0) (at 133.985 118.7449 0)
-      (effects (font (size 1.27 1.27)) (justify right))
-    )
-    (property "Value" "2.2uF" (id 1) (at 133.985 121.2849 0)
-      (effects (font (size 1.27 1.27)) (justify right))
-    )
-    (property "Footprint" "Capacitor_SMD:C_0805_2012Metric" (id 2) (at 138.7602 116.205 0)
-      (effects (font (size 1.27 1.27)) hide)
-    )
-    (property "Datasheet" "~" (id 3) (at 137.795 120.015 0)
-      (effects (font (size 1.27 1.27)) hide)
-    )
-    (property "JLCPCB" "C49217" (id 4) (at 137.795 120.015 0)
-      (effects (font (size 1.27 1.27)) hide)
-    )
-    (pin "1")
-    (pin "2")
-  )
-  (symbol (lib_id "power:GNDD") (at 142.875 123.825 0) (unit 1)
-    (in_bom yes) (on_board yes)
-    (property "Reference" "#PWR049" (id 0) (at 142.875 130.175 0)
-      (effects (font (size 1.27 1.27)) hide)
-    )
-    (property "Value" "GNDD" (id 1) (at 140.335 127.635 0)
-      (effects (font (size 1.27 1.27)) (justify left))
-    )
-    (property "Footprint" "" (id 2) (at 142.875 123.825 0)
-      (effects (font (size 1.27 1.27)) hide)
-    )
-    (property "Datasheet" "" (id 3) (at 142.875 123.825 0)
+  (symbol (lib_id "power:GNDD") (at 138.43 123.825 0) (unit 1)
+    (in_bom yes) (on_board yes)
+    (property "Reference" "#PWR049" (id 0) (at 138.43 130.175 0)
+      (effects (font (size 1.27 1.27)) hide)
+    )
+    (property "Value" "GNDD" (id 1) (at 135.89 127.635 0)
+      (effects (font (size 1.27 1.27)) (justify left))
+    )
+    (property "Footprint" "" (id 2) (at 138.43 123.825 0)
+      (effects (font (size 1.27 1.27)) hide)
+    )
+    (property "Datasheet" "" (id 3) (at 138.43 123.825 0)
       (effects (font (size 1.27 1.27)) hide)
     )
@@
       (effects (font (size 1.27 1.27)) hide)
     )
-    (property "JLCPCB" "C25744" (id 4) (at 140.335 66.675 0)
+    (property "JLCPCB" "" (id 4) (at 140.335 66.675 0)
+      (effects (font (size 1.27 1.27)) hide)
+    )
+    (property "LCSC" "C25744" (id 5) (at 140.335 66.675 0)
       (effects (font (size 1.27 1.27)) hide)
     )
     (pin "1")
     (pin "2")
-  )
-  (symbol (lib_id "power:GNDD") (at 137.795 123.825 0) (unit 1)
-    (in_bom yes) (on_board yes)
-    (property "Reference" "#PWR047" (id 0) (at 137.795 130.175 0)
-      (effects (font (size 1.27 1.27)) hide)
-    )
-    (property "Value" "GNDD" (id 1) (at 135.255 127.635 0)
-      (effects (font (size 1.27 1.27)) (justify left))
-    )
-    (property "Footprint" "" (id 2) (at 137.795 123.825 0)
-      (effects (font (size 1.27 1.27)) hide)
-    )
-    (property "Datasheet" "" (id 3) (at 137.795 123.825 0)
-      (effects (font (size 1.27 1.27)) hide)
-    )
-    (pin "1")
   )
   (symbol (lib_id "power:VBUS") (at 154.94 64.135 0) (unit 1)
@@
       (effects (font (size 1.27 1.27)) hide)
     )
+    (property "LCSC" "C25905" (id 5) (at 106.68 81.28 90)
+      (effects (font (size 1.27 1.27)) hide)
+    )
     (pin "1")
     (pin "2")
   )
-  (symbol (lib_id "Device:C") (at 142.875 120.015 0) (mirror x) (unit 1)
-    (in_bom yes) (on_board yes)
-    (property "Reference" "C10" (id 0) (at 146.05 118.11 0)
-      (effects (font (size 1.27 1.27)) (justify right))
-    )
-    (property "Value" "2.2uF" (id 1) (at 149.225 122.555 0)
-      (effects (font (size 1.27 1.27)) (justify right))
-    )
-    (property "Footprint" "Capacitor_SMD:C_0805_2012Metric" (id 2) (at 143.8402 116.205 0)
-      (effects (font (size 1.27 1.27)) hide)
-    )
-    (property "Datasheet" "~" (id 3) (at 142.875 120.015 0)
-      (effects (font (size 1.27 1.27)) hide)
-    )
-    (property "JLCPCB" "C49217" (id 4) (at 142.875 120.015 0)
+  (symbol (lib_id "Device:C") (at 138.43 120.015 0) (unit 1)
+    (in_bom yes) (on_board yes)
+    (property "Reference" "C7" (id 0) (at 142.24 118.7449 0)
+      (effects (font (size 1.27 1.27)) (justify left))
+    )
+    (property "Value" "47uF" (id 1) (at 142.24 121.2849 0)
+      (effects (font (size 1.27 1.27)) (justify left))
+    )
+    (property "Footprint" "Capacitor_SMD:C_0805_2012Metric" (id 2) (at 139.3952 123.825 0)
+      (effects (font (size 1.27 1.27)) hide)
+    )
+    (property "Datasheet" "~" (id 3) (at 138.43 120.015 0)
+      (effects (font (size 1.27 1.27)) hide)
+    )
+    (property "JLCPCB" "" (id 4) (at 138.43 120.015 0)
+      (effects (font (size 1.27 1.27)) hide)
+    )
+    (property "LCSC" "C16780" (id 5) (at 138.43 120.015 0)
       (effects (font (size 1.27 1.27)) hide)
     )
@@
     )
     (pin "1")
-  )
-  (symbol (lib_id "Device:C") (at 124.46 120.015 0) (mirror x) (unit 1)
-    (in_bom yes) (on_board yes) (fields_autoplaced)
-    (property "Reference" "C4" (id 0) (at 120.65 118.7449 0)
-      (effects (font (size 1.27 1.27)) (justify right))
-    )
-    (property "Value" "2.2uF" (id 1) (at 120.65 121.2849 0)
-      (effects (font (size 1.27 1.27)) (justify right))
-    )
-    (property "Footprint" "Capacitor_SMD:C_0805_2012Metric" (id 2) (at 125.4252 116.205 0)
-      (effects (font (size 1.27 1.27)) hide)
-    )
-    (property "Datasheet" "~" (id 3) (at 124.46 120.015 0)
-      (effects (font (size 1.27 1.27)) hide)
-    )
-    (property "JLCPCB" "C49217" (id 4) (at 124.46 120.015 0)
-      (effects (font (size 1.27 1.27)) hide)
-    )
-    (pin "1")
-    (pin "2")
   )
   (symbol (lib_id "Device:R_US") (at 106.68 83.82 90) (unit 1)
@@
       (effects (font (size 1.27 1.27)) hide)
     )
+    (property "LCSC" "C25905" (id 5) (at 106.68 83.82 90)
+      (effects (font (size 1.27 1.27)) hide)
+    )
+    (pin "1")
+    (pin "2")
+  )
+  (symbol (lib_id "Device:C") (at 124.46 120.015 0) (unit 1)
+    (in_bom yes) (on_board yes)
+    (property "Reference" "C4" (id 0) (at 128.27 118.7449 0)
+      (effects (font (size 1.27 1.27)) (justify left))
+    )
+    (property "Value" "47uF" (id 1) (at 128.27 121.2849 0)
+      (effects (font (size 1.27 1.27)) (justify left))
+    )
+    (property "Footprint" "Capacitor_SMD:C_0805_2012Metric" (id 2) (at 125.4252 123.825 0)
+      (effects (font (size 1.27 1.27)) hide)
+    )
+    (property "Datasheet" "~" (id 3) (at 124.46 120.015 0)
+      (effects (font (size 1.27 1.27)) hide)
+    )
+    (property "JLCPCB" "" (id 4) (at 124.46 120.015 0)
+      (effects (font (size 1.27 1.27)) hide)
+    )
+    (property "LCSC" "C16780" (id 5) (at 124.46 120.015 0)
+      (effects (font (size 1.27 1.27)) hide)
+    )
