File: hw/pcb/OrbitESC/USB2Serial.kicad_sch (KiCad schematic)
At the start: 12 parts, among them J1 USB_C_Receptacle_USB2.0, U10 CP2104

Commit message: Squash feature/sync_current_ctrl/r0
Parts:
- removed C10: 2.2uF, Capacitor_SMD:C_0805_2012Metric, symbol Device:C
- removed D6, D7: Yellow LED, Diode_SMD:D_0603_1608Metric, symbol Device:LED
- removed R19, R20: 1.5k, Resistor_SMD:R_0402_1005Metric, symbol Device:R_US
- C4, C7: value 2.2uF -> 47uF; JLCPCB C49217 -> (none); LCSC (none) -> C16780
- R13, R9: LCSC (none) -> C25905
- R15: JLCPCB C25744 -> (none); LCSC (none) -> C25744
Connections:
- net GNDD: now also C4.2, C7.2; no longer C4.1, C7.1
- net VBUS: now also C4.1; no longer C4.2
- net at U10.16 (VPP): now also C7.1; no longer C7.2
- no-connect marks 13 -> 15
