File: hw/pcb/OrbitESC/power_supply.kicad_sch (KiCad schematic)
At the start: 30 parts, among them J11 VDC, J12 GND, Q7 2N7002, U7 AP62200Z6-7, U8 AP2171W, U9 AP2120

Commit message: Finalize V2 PCB
Parts:
- C22, C24, C28, C34, C36: JLCPCB C307331 -> (none); LCSC (none) -> C307331
- C23: JLCPCB C440198 -> (none); LCSC (none) -> C440198
- C25, C26: JLCPCB C16780 -> (none); LCSC (none) -> C16780
- C27, C29, C33: JLCPCB C49217 -> (none); LCSC (none) -> C49217
- D1: JLCPCB C72041 -> (none); LCSC (none) -> C72041
- D8: JLCPCB C8598 -> (none); LCSC (none) -> C8598
- FB1: JLCPCB C1002 -> (none); LCSC (none) -> C1002
- Q7: JLCPCB C8545 -> (none); LCSC (none) -> C8545
- R37, R38, R41, R43, R44: JLCPCB C25744 -> (none); LCSC (none) -> C25744
- R39: JLCPCB C11702 -> (none); LCSC (none) -> C11702
- R40: JLCPCB C25796 -> (none); LCSC (none) -> C25796
- R42: JLCPCB C25077 -> (none); LCSC (none) -> C25077
- U7: LCSC (none) -> C2158024
Changed lines of the file:
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@@
       (effects (font (size 1.27 1.27)) hide)
     )
-    (property "JLCPCB" "C25744" (id 4) (at 125.73 48.895 0)
+    (property "JLCPCB" "" (id 4) (at 125.73 48.895 0)
+      (effects (font (size 1.27 1.27)) hide)
+    )
+    (property "LCSC" "C25744" (id 5) (at 125.73 48.895 0)
       (effects (font (size 1.27 1.27)) hide)
     )
@@
       (effects (font (size 1.27 1.27)) hide)
     )
-    (property "JLCPCB" "C25796" (id 4) (at 176.53 52.705 0)
+    (property "JLCPCB" "" (id 4) (at 176.53 52.705 0)
       (effects (font (size 1.27 1.27)) hide)
     )
     (property "DigiKey" "RMCF0402FT57K6CT-ND" (id 5) (at 176.53 52.705 0)
+      (effects (font (size 1.27 1.27)) hide)
+    )
+    (property "LCSC" "C25796" (id 6) (at 176.53 52.705 0)
       (effects (font (size 1.27 1.27)) hide)
     )
@@
       (effects (font (size 1.27 1.27)) hide)
     )
-    (property "JLCPCB" "C8598" (id 4) (at 217.17 46.355 0)
+    (property "JLCPCB" "" (id 4) (at 217.17 46.355 0)
+      (effects (font (size 1.27 1.27)) hide)
+    )
+    (property "LCSC" "C8598" (id 5) (at 217.17 46.355 0)
       (effects (font (size 1.27 1.27)) hide)
     )
@@
     )
     (property "DigiKey" "31-AP62200Z6-7CT-ND" (id 4) (at 142.24 46.355 0)
+      (effects (font (size 1.27 1.27)) hide)
+    )
+    (property "LCSC" "C2158024" (id 5) (at 142.24 46.355 0)
       (effects (font (size 1.27 1.27)) hide)
     )
@@
       (effects (font (size 1.27 1.27)) hide)
     )
-    (property "JLCPCB" "C25077" (id 4) (at 179.705 106.68 90)
+    (property "JLCPCB" "" (id 4) (at 179.705 106.68 90)
+      (effects (font (size 1.27 1.27)) hide)
+    )
+    (property "LCSC" "C25077" (id 5) (at 179.705 106.68 0)
       (effects (font (size 1.27 1.27)) hide)
     )
@@
       (effects (font (size 1.27 1.27)) hide)
     )
-    (property "JLCPCB" "C25744" (id 4) (at 72.39 51.435 0)
+    (property "JLCPCB" "" (id 4) (at 72.39 51.435 0)
+      (effects (font (size 1.27 1.27)) hide)
+    )
+    (property "LCSC" "C25744" (id 5) (at 72.39 51.435 0)
       (effects (font (size 1.27 1.27)) hide)
     )
@@
       (effects (font (size 1.27 1.27)) hide)
     )
-    (property "JLCPCB" "C307331" (id 4) (at 165.1 115.57 0)
+    (property "JLCPCB" "" (id 4) (at 165.1 115.57 0)
+      (effects (font (size 1.27 1.27)) hide)
+    )
+    (property "LCSC" "C307331" (id 5) (at 165.1 115.57 0)
       (effects (font (size 1.27 1.27)) hide)
     )
@@
       (effects (font (size 1.27 1.27)) (justify left) hide)
     )
-    (property "JLCPCB" "C8545" (id 4) (at 103.505 120.65 0)
+    (property "JLCPCB" "" (id 4) (at 103.505 120.65 0)
+      (effects (font (size 1.27 1.27)) hide)
+    )
+    (property "LCSC" "C8545" (id 5) (at 103.505 120.65 0)
       (effects (font (size 1.27 1.27)) hide)
     )
@@
       (effects (font (size 1.27 1.27)) hide)
     )
-    (property "JLCPCB" "C307331" (id 4) (at 191.135 115.57 0)
+    (property "JLCPCB" "" (id 4) (at 191.135 115.57 0)
+      (effects (font (size 1.27 1.27)) hide)
+    )
+    (property "LCSC" "C307331" (id 5) (at 191.135 115.57 0)
       (effects (font (size 1.27 1.27)) hide)
     )
@@
       (effects (font (size 1.27 1.27)) hide)
     )
-    (property "JLCPCB" "C307331" (id 4) (at 102.87 57.785 0)
+    (property "JLCPCB" "" (id 4) (at 102.87 57.785 0)
+      (effects (font (size 1.27 1.27)) hide)
+    )
+    (property "LCSC" "C307331" (id 5) (at 102.87 57.785 0)
       (effects (font (size 1.27 1.27)) hide)
     )
@@
       (effects (font (size 1.27 1.27)) hide)
     )
-    (property "JLCPCB" "C49217" (id 4) (at 158.75 115.57 0)
+    (property "JLCPCB" "" (id 4) (at 158.75 115.57 0)
+      (effects (font (size 1.27 1.27)) hide)
+    )
+    (property "LCSC" "C49217" (id 5) (at 158.75 115.57 0)
       (effects (font (size 1.27 1.27)) hide)
     )
@@
       (effects (font (size 1.27 1.27)) hide)
     )
-    (property "JLCPCB" "C72041" (id 4) (at 72.39 61.595 90)
+    (property "JLCPCB" "" (id 4) (at 72.39 61.595 90)
+      (effects (font (size 1.27 1.27)) hide)
+    )
+    (property "LCSC" "C72041" (id 5) (at 72.39 61.595 0)
       (effects (font (size 1.27 1.27)) hide)
     )
@@
       (effects (font (size 1.27 1.27)) hide)
     )
-    (property "JLCPCB" "C307331" (id 4) (at 158.75 46.355 0)
+    (property "JLCPCB" "" (id 4) (at 158.75 46.355 0)
+      (effects (font (size 1.27 1.27)) hide)
+    )
+    (property "LCSC" "C307331" (id 5) (at 158.75 46.355 0)
       (effects (font (size 1.27 1.27)) hide)
     )
@@
       (effects (font (size 1.27 1.27)) hide)
     )
-    (property "JLCPCB" "C16780" (id 4) (at 198.12 57.785 0)
+    (property "JLCPCB" "" (id 4) (at 198.12 57.785 0)
+      (effects (font (size 1.27 1.27)) hide)
+    )
+    (property "LCSC" "C16780" (id 5) (at 198.12 57.785 0)
       (effects (font (size 1.27 1.27)) hide)
     )
@@
       (effects (font (size 1.27 1.27)) hide)
     )
-    (property "JLCPCB" "C16780" (id 4) (at 209.55 57.785 0)
+    (property "JLCPCB" "" (id 4) (at 209.55 57.785 0)
+      (effects (font (size 1.27 1.27)) hide)
+    )
+    (property "LCSC" "C16780" (id 5) (at 209.55 57.785 0)
       (effects (font (size 1.27 1.27)) hide)
     )
@@
       (effects (font (size 1.27 1.27)) hide)
     )
-    (property "JLCPCB" "C1002" (id 4) (at 169.545 106.68 90)
+    (property "JLCPCB" "" (id 4) (at 169.545 106.68 90)
+      (effects (font (size 1.27 1.27)) hide)
+    )
+    (property "LCSC" "C1002" (id 5) (at 169.545 106.68 0)
       (effects (font (size 1.27 1.27)) hide)
     )
@@
       (effects (font (size 1.27 1.27)) hide)
     )
-    (property "JLCPCB" "C49217" (id 4) (at 133.35 115.57 0)
+    (property "JLCPCB" "" (id 4) (at 133.35 115.57 0)
+      (effects (font (size 1.27 1.27)) hide)
+    )
+    (property "LCSC" "C49217" (id 5) (at 133.35 115.57 0)
       (effects (font (size 1.27 1.27)) hide)
     )
@@
       (effects (font (size 1.27 1.27)) hide)
     )
-    (property "JLCPCB" "C25744" (id 4) (at 100.965 111.76 0)
+    (property "JLCPCB" "" (id 4) (at 100.965 111.76 0)
+      (effects (font (size 1.27 1.27)) hide)
+    )
+    (property "LCSC" "C25744" (id 5) (at 100.965 111.76 0)
       (effects (font (size 1.27 1.27)) hide)
     )
@@
       (effects (font (size 1.27 1.27)) hide)
     )
-    (property "JLCPCB" "C25744" (id 4) (at 176.53 62.865 0)
+    (property "JLCPCB" "" (id 4) (at 176.53 62.865 0)
+      (effects (font (size 1.27 1.27)) hide)
+    )
+    (property "LCSC" "C25744" (id 5) (at 176.53 62.865 0)
       (effects (font (size 1.27 1.27)) hide)
     )
@@
       (effects (font (size 1.27 1.27)) hide)
     )
-    (property "JLCPCB" "C49217" (id 4) (at 184.785 115.57 0)
+    (property "JLCPCB" "" (id 4) (at 184.785 115.57 0)
+      (effects (font (size 1.27 1.27)) hide)
+    )
+    (property "LCSC" "C49217" (id 5) (at 184.785 115.57 0)
       (effects (font (size 1.27 1.27)) hide)
     )
@@
       (effects (font (size 1.27 1.27)) hide)
     )
-    (property "JLCPCB" "C25744" (id 4) (at 95.885 127 0)
+    (property "JLCPCB" "" (id 4) (at 95.885 127 0)
+      (effects (font (size 1.27 1.27)) hide)
+    )
+    (property "LCSC" "C25744" (id 5) (at 95.885 127 0)
       (effects (font (size 1.27 1.27)) hide)
     )
@@
       (effects (font (size 1.27 1.27)) hide)
     )
-    (property "JLCPCB" "C307331" (id 4) (at 185.42 57.785 0)
+    (property "JLCPCB" "" (id 4) (at 185.42 57.785 0)
+      (effects (font (size 1.27 1.27)) hide)
+    )
+    (property "LCSC" "C307331" (id 5) (at 185.42 57.785 0)
       (effects (font (size 1.27 1.27)) hide)
     )
@@
       (effects (font (size 1.27 1.27)) hide)
     )
-    (property "JLCPCB" "C440198" (id 4) (at 109.22 57.785 0)
+    (property "JLCPCB" "" (id 4) (at 109.22 57.785 0)
+      (effects (font (size 1.27 1.27)) hide)
+    )
+    (property "LCSC" "C440198" (id 5) (at 109.22 57.785 0)
       (effects (font (size 1.27 1.27)) hide)
     )
@@
       (effects (font (size 1.27 1.27)) hide)
     )
-    (property "JLCPCB" "C11702" (id 4) (at 90.805 120.65 0)
-      (effects (font (size 1.27 1.27)) hide)
-    )
+    (property "JLCPCB" "" (id 4) (at 90.805 120.65 0)
+      (effects (font (size 1.27 1.27)) hide)
+    )
+    (property "LCSC" "C11702" (id 5) (at 90.805 120.65 0)
+      (effects (font (size 1.27 1.27)) hide)
+    )
