File: hw/pcb/OrbitESC_V3/status_leds.kicad_sch (KiCad schematic)
At the start: 18 parts, among them U12 74HC595BQ

Commit message: Sync board design
Parts:
- removed D16, D17, D19: Blue LED, Diode_SMD:D_0603_1608Metric, symbol Device:LED
- removed R87, R88, R90: 470, Resistor_SMD:R_0402_1005Metric, symbol Device:R_US
Connections:
- net STATUS_0 is gone; now on net HEARTBEAT: U12.4 (QE)
- net STATUS_1 is gone; now on net CAN1_ACTV: U12.5 (QF)
- net ARMED: now also U12.3 (QD); no longer U12.1 (QB)
- net CAN1_ACTV: no longer U12.3 (QD)
- net FAULT: now also U12.2 (QC); no longer U12.15 (QA)
- net HEARTBEAT: no longer U12.2 (QC)
- net STATUS_2: no longer names the net of U12.6 (QG)
- no-connect marks 2 -> 5
