File: hw/pcb/OrbitESC_V3/microcontroller.kicad_sch (KiCad schematic)
At the start: 29 parts, among them J6 CAN1, SW1 Reset, U1 TLE9250X, U11 STM32L432KCU6, U2 AT25SF128A-SHB-T

Commit message: save pcb work
Parts:
- removed J6: CAN1, Connector_JST:JST_PH_B3B-PH-K_1x03_P2.00mm_Vertical, symbol Connector:Conn_01x03_Male
- added J11: RX, TestPoint:TestPoint_Pad_1.5x1.5mm, symbol Connector:Conn_01x01_Female
- added J11: CANH, TestPoint:TestPoint_Pad_1.5x1.5mm, symbol Connector:Conn_01x01_Female
- added J11: GND, TestPoint:TestPoint_Pad_1.5x1.5mm, symbol Connector:Conn_01x01_Female
- added J11: TX, TestPoint:TestPoint_Pad_1.5x1.5mm, symbol Connector:Conn_01x01_Female
- added J11: CANL, TestPoint:TestPoint_Pad_1.5x1.5mm, symbol Connector:Conn_01x01_Female
Connections:
- net GND: now also J11.1 (Pin_1)
- net SERIAL1_IN: now also J11.1 (Pin_1)
- net SERIAL1_OUT: now also J11.1 (Pin_1)
- net at R62.1, U1.6 (CANL): now also J11.1 (Pin_1)
- net at R62.2, U1.7 (CANH): now also J11.1 (Pin_1)
Changed lines of the file:
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@@
   (junction (at 199.39 172.72) (diameter 0) (color 0 0 0 0)
   )
+  (junction (at 120.65 123.19) (diameter 0) (color 0 0 0 0)
+  )
   (junction (at 210.185 66.04) (diameter 0) (color 0 0 0 0)
+  )
+  (junction (at 124.46 118.745) (diameter 0) (color 0 0 0 0)
   )
   (junction (at 255.905 157.48) (diameter 0) (color 0 0 0 0)
@@
     (stroke (width 0) (type default))
   )
-  (wire (pts (xy 99.695 118.745) (xy 104.775 118.745))
+  (wire (pts (xy 99.695 118.745) (xy 124.46 118.745))
     (stroke (width 0) (type default))
   )
@@
     (stroke (width 0) (type default))
   )
-  (wire (pts (xy 99.695 123.19) (xy 104.775 123.19))
+  (wire (pts (xy 99.695 123.19) (xy 120.65 123.19))
     (stroke (width 0) (type default))
   )
@@
     (stroke (width 0) (type default))
   )
+  (wire (pts (xy 124.46 116.84) (xy 124.46 118.745))
+    (stroke (width 0) (type default))
+  )
   (wire (pts (xy 210.185 52.07) (xy 210.185 53.34))
     (stroke (width 0) (type default))
@@
     (stroke (width 0) (type default))
   )
+  (wire (pts (xy 124.46 118.745) (xy 128.905 118.745))
+    (stroke (width 0) (type default))
+  )
+  (wire (pts (xy 120.65 123.19) (xy 128.905 123.19))
+    (stroke (width 0) (type default))
+  )
   (wire (pts (xy 252.73 53.34) (xy 259.08 53.34))
     (stroke (width 0) (type default))
@@
   )
   (wire (pts (xy 134.62 163.195) (xy 134.62 159.385))
+    (stroke (width 0) (type default))
+  )
+  (wire (pts (xy 120.65 116.84) (xy 120.65 123.19))
     (stroke (width 0) (type default))
   )
@@
     )
   )
-  (global_label "SERIAL1_OUT" (shape input) (at 104.775 118.745 0) (fields_autoplaced)
-    (effects (font (size 1.27 1.27)) (justify left))
-    (property "Intersheetrefs" "${INTERSHEET_REFS}" (at 119.3438 118.6656 0)
+  (global_label "SERIAL1_OUT" (shape input) (at 128.905 118.745 0) (fields_autoplaced)
+    (effects (font (size 1.27 1.27)) (justify left))
+    (property "Intersheetrefs" "${INTERSHEET_REFS}" (at 143.4738 118.6656 0)
       (effects (font (size 1.27 1.27)) (justify left) hide)
     )
@@
     )
   )
-  (global_label "SERIAL1_IN" (shape output) (at 104.775 123.19 0) (fields_autoplaced)
-    (effects (font (size 1.27 1.27)) (justify left))
-    (property "Intersheetrefs" "${INTERSHEET_REFS}" (at 117.6505 123.1106 0)
+  (global_label "SERIAL1_IN" (shape output) (at 128.905 123.19 0) (fields_autoplaced)
+    (effects (font (size 1.27 1.27)) (justify left))
+    (property "Intersheetrefs" "${INTERSHEET_REFS}" (at 141.7805 123.1106 0)
       (effects (font (size 1.27 1.27)) (justify left) hide)
     )
@@
     )
   )
+  (symbol (lib_id "Connector:Conn_01x01_Female") (at 120.65 111.76 90) (unit 1)
+    (in_bom yes) (on_board yes) (dnp no)
+    (property "Reference" "J11" (at 119.8153 111.0488 0)
+      (effects (font (size 1.27 1.27)) (justify left))
+    )
+    (property "Value" "RX" (at 120.65 108.585 0)
+      (effects (font (size 1.27 1.27)) (justify left))
+    )
+    (property "Footprint" "TestPoint:TestPoint_Pad_1.5x1.5mm" (at 120.65 111.76 0)
+      (effects (font (size 1.27 1.27)) hide)
+    )
+    (property "Datasheet" "~" (at 120.65 111.76 0)
+      (effects (font (size 1.27 1.27)) hide)
+    )
+    (property "DigiKey" "N/A" (at 120.65 111.76 0)
+      (effects (font (size 1.27 1.27)) hide)
+    )
+    (pin "1")
+    (instances
+      (project "OrbitESC"
+        (path "/a13534e1-2c37-4692-a99c-4eada4007967/e5c7e094-5305-4041-9a38-3256d4457e28"
+          (reference "J11") (unit 1)
+        )
+        (path "/a13534e1-2c37-4692-a99c-4eada4007967/ed067bb8-caa7-448e-917b-cc2d33c8b4b7"
+          (reference "J8") (unit 1)
+        )
+        (path "/a13534e1-2c37-4692-a99c-4eada4007967/ed067bb8-caa7-448e-917b-cc2d33c8b4b7/6349e373-ae96-42f5-b0a0-1a23031b19cc"
+          (reference "J8") (unit 1)
+        )
+      )
+    )
+  )
   (symbol (lib_id "power:GNDD") (at 204.47 109.22 0) (unit 1)
     (in_bom yes) (on_board yes) (dnp no)
@@
         (path "/a13534e1-2c37-4692-a99c-4eada4007967/ed067bb8-caa7-448e-917b-cc2d33c8b4b7"
           (reference "#PWR0124") (unit 1)
+        )
+      )
+    )
+  )
+  (symbol (lib_id "Connector:Conn_01x01_Female") (at 140.97 154.305 0) (unit 1)
+    (in_bom yes) (on_board yes) (dnp no)
+    (property "Reference" "J11" (at 141.6812 153.4703 0)
+      (effects (font (size 1.27 1.27)) (justify left))
+    )
+    (property "Value" "CANH" (at 144.145 154.305 0)
+      (effects (font (size 1.27 1.27)) (justify left))
+    )
+    (property "Footprint" "TestPoint:TestPoint_Pad_1.5x1.5mm" (at 140.97 154.305 0)
+      (effects (font (size 1.27 1.27)) hide)
+    )
+    (property "Datasheet" "~" (at 140.97 154.305 0)
+      (effects (font (size 1.27 1.27)) hide)
+    )
+    (property "DigiKey" "N/A" (at 140.97 154.305 0)
+      (effects (font (size 1.27 1.27)) hide)
+    )
+    (pin "1")
+    (instances
+      (project "OrbitESC"
+        (path "/a13534e1-2c37-4692-a99c-4eada4007967/e5c7e094-5305-4041-9a38-3256d4457e28"
+          (reference "J11") (unit 1)
+        )
+        (path "/a13534e1-2c37-4692-a99c-4eada4007967/ed067bb8-caa7-448e-917b-cc2d33c8b4b7"
+          (reference "J2") (unit 1)
         )
       )
@@
     )
   )
+  (symbol (lib_id "Connector:Conn_01x01_Female") (at 140.97 156.845 0) (unit 1)
+    (in_bom yes) (on_board yes) (dnp no)
+    (property "Reference" "J11" (at 141.6812 156.0103 0)
+      (effects (font (size 1.27 1.27)) (justify left))
+    )
+    (property "Value" "GND" (at 144.145 156.845 0)
+      (effects (font (size 1.27 1.27)) (justify left))
+    )
+    (property "Footprint" "TestPoint:TestPoint_Pad_1.5x1.5mm" (at 140.97 156.845 0)
+      (effects (font (size 1.27 1.27)) hide)
+    )
+    (property "Datasheet" "~" (at 140.97 156.845 0)
+      (effects (font (size 1.27 1.27)) hide)
+    )
+    (property "DigiKey" "N/A" (at 140.97 156.845 0)
+      (effects (font (size 1.27 1.27)) hide)
+    )
+    (pin "1")
+    (instances
+      (project "OrbitESC"
+        (path "/a13534e1-2c37-4692-a99c-4eada4007967/e5c7e094-5305-4041-9a38-3256d4457e28"
+          (reference "J11") (unit 1)
+        )
+        (path "/a13534e1-2c37-4692-a99c-4eada4007967/ed067bb8-caa7-448e-917b-cc2d33c8b4b7"
+          (reference "J6") (unit 1)
+        )
+      )
+    )
+  )
   (symbol (lib_id "Device:C") (at 204.47 105.41 180) (unit 1)
     (in_bom yes) (on_board yes) (dnp no)
@@
     )
   )
+  (symbol (lib_id "Connector:Conn_01x01_Female") (at 124.46 111.76 90) (unit 1)
+    (in_bom yes) (on_board yes) (dnp no)
+    (property "Reference" "J11" (at 123.6253 111.0488 0)
+      (effects (font (size 1.27 1.27)) (justify left))
+    )
+    (property "Value" "TX" (at 124.46 108.585 0)
+      (effects (font (size 1.27 1.27)) (justify left))
+    )
+    (property "Footprint" "TestPoint:TestPoint_Pad_1.5x1.5mm" (at 124.46 111.76 0)
+      (effects (font (size 1.27 1.27)) hide)
+    )
+    (property "Datasheet" "~" (at 124.46 111.76 0)
+      (effects (font (size 1.27 1.27)) hide)
+    )
+    (property "DigiKey" "N/A" (at 124.46 111.76 0)
+      (effects (font (size 1.27 1.27)) hide)
+    )
+    (pin "1")
+    (instances
+      (project "OrbitESC"
+        (path "/a13534e1-2c37-4692-a99c-4eada4007967/e5c7e094-5305-4041-9a38-3256d4457e28"
+          (reference "J11") (unit 1)
+        )
+        (path "/a13534e1-2c37-4692-a99c-4eada4007967/ed067bb8-caa7-448e-917b-cc2d33c8b4b7"
+          (reference "J9") (unit 1)
+        )
+        (path "/a13534e1-2c37-4692-a99c-4eada4007967/ed067bb8-caa7-448e-917b-cc2d33c8b4b7/6349e373-ae96-42f5-b0a0-1a23031b19cc"
+          (reference "J9") (unit 1)
+        )
+      )
+    )
+  )
   (symbol (lib_id "power:GNDD") (at 210.185 67.31 0) (unit 1)
     (in_bom yes) (on_board yes) (dnp no)
@@
     )
   )
+  (symbol (lib_id "Connector:Conn_01x01_Female") (at 140.97 159.385 0) (unit 1)
+    (in_bom yes) (on_board yes) (dnp no)
+    (property "Reference" "J11" (at 141.6812 158.5503 0)
+      (effects (font (size 1.27 1.27)) (justify left))
+    )
+    (property "Value" "CANL" (at 144.145 159.385 0)
+      (effects (font (size 1.27 1.27)) (justify left))
+    )
+    (property "Footprint" "TestPoint:TestPoint_Pad_1.5x1.5mm" (at 140.97 159.385 0)
+      (effects (font (size 1.27 1.27)) hide)
+    )
+    (property "Datasheet" "~" (at 140.97 159.385 0)
+      (effects (font (size 1.27 1.27)) hide)
+    )
+    (property "DigiKey" "N/A" (at 140.97 159.385 0)
+      (effects (font (size 1.27 1.27)) hide)
+    )
+    (pin "1")
+    (instances
+      (project "OrbitESC"
+        (path "/a13534e1-2c37-4692-a99c-4eada4007967/e5c7e094-5305-4041-9a38-3256d4457e28"
+          (reference "J11") (unit 1)
+        )
+        (path "/a13534e1-2c37-4692-a99c-4eada4007967/ed067bb8-caa7-448e-917b-cc2d33c8b4b7"
+          (reference "J7") (unit 1)
+        )
+      )
+    )
+  )
   (symbol (lib_id "Device:R_US") (at 259.08 58.42 180) (unit 1)
     (in_bom yes) (on_board yes) (dnp no) (fields_autoplaced)
@@
         )
       )
-    )
-  )
-  (symbol (lib_id "Connector:Conn_01x03_Male") (at 140.97 156.845 0) (mirror y) (unit 1)
-    (in_bom yes) (on_board yes) (dnp no) (fields_autoplaced)
-    (property "Reference" "J6" (at 142.24 155.5749 0)
-      (effects (font (size 1.27 1.27)) (justify right))
-    )
-    (property "Value" "CAN1" (at 142.24 158.1149 0)
-      (effects (font (size 1.27 1.27)) (justify right))
-    )
-    (property "Footprint" "Connector_JST:JST_PH_B3B-PH-K_1x03_P2.00mm_Vertical" (at 140.97 156.845 0)
-      (effects (font (size 1.27 1.27)) hide)
-    )
-    (property "Datasheet" "~" (at 140.97 156.845 0)
-      (effects (font (size 1.27 1.27)) hide)
-    )
-    (property "DigiKey" "A100035-ND" (at 140.97 156.845 0)
-      (effects (font (size 1.27 1.27)) hide)
-    )
-    (pin "1")
-    (pin "2")
-    (pin "3")
-    (instances
-      (project "OrbitESC"
-        (path "/a13534e1-2c37-4692-a99c-4eada4007967/ed067bb8-caa7-448e-917b-cc2d33c8b4b7"
-          (reference "J6") (unit 1)
-        )
-      )

Commit message: Lazy sync for work over the past few weeks. Been busy
Parts:
- added J13: Micro_SD_Card, symbol Connector:Micro_SD_Card
- added U3: STM32F446RETx, Package_QFP:LQFP-64_10x10mm_P0.5mm, symbol MCU_ST_STM32F4:STM32F446RETx
Connections:
- new net: U3.18 (VSS), U3.31 (VSS), U3.47 (VSS), U3.63 (VSS)
Other:
- note added: "Keep both SPI and SD card for now"
Changed lines of the file:
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@@
+    (effects (font (size 1.27 1.27)) (justify left bottom))
+  )
+  (text "Keep both SPI and SD card for now" (at 243.84 177.165 0)
     (effects (font (size 1.27 1.27)) (justify left bottom))
   )
@@
     )
   )
+  (symbol (lib_id "MCU_ST_STM32F4:STM32F446RETx") (at 172.085 228.6 0) (unit 1)
+    (in_bom yes) (on_board yes) (dnp no) (fields_autoplaced)
+    (property "Reference" "U3" (at 176.5809 274.32 0)
+      (effects (font (size 1.27 1.27)) (justify left))
+    )
+    (property "Value" "STM32F446RETx" (at 176.5809 276.86 0)
+      (effects (font (size 1.27 1.27)) (justify left))
+    )
+    (property "Footprint" "Package_QFP:LQFP-64_10x10mm_P0.5mm" (at 156.845 271.78 0)
+      (effects (font (size 1.27 1.27)) (justify right) hide)
+    )
+    (property "Datasheet" "https://www.st.com/resource/en/datasheet/stm32f446re.pdf" (at 172.085 228.6 0)
+      (effects (font (size 1.27 1.27)) hide)
+    )
+    (pin "1")
+    (pin "10")
+    (pin "11")
+    (pin "12")
+    (pin "13")
+    (pin "14")
+    (pin "15")
+    (pin "16")
+    (pin "17")
+    (pin "18")
+    (pin "19")
+    (pin "2")
+    (pin "20")
+    (pin "21")
+    (pin "22")
+    (pin "23")
+    (pin "24")
+    (pin "25")
+    (pin "26")
+    (pin "27")
+    (pin "28")
+    (pin "29")
+    (pin "3")
+    (pin "30")
+    (pin "31")
+    (pin "32")
+    (pin "33")
+    (pin "34")
+    (pin "35")
+    (pin "36")
+    (pin "37")
+    (pin "38")
+    (pin "39")
+    (pin "4")
+    (pin "40")
+    (pin "41")
+    (pin "42")
+    (pin "43")
+    (pin "44")
+    (pin "45")
+    (pin "46")
+    (pin "47")
+    (pin "48")
+    (pin "49")
+    (pin "5")
+    (pin "50")
+    (pin "51")
+    (pin "52")
+    (pin "53")
+    (pin "54")
+    (pin "55")
+    (pin "56")
+    (pin "57")
+    (pin "58")
+    (pin "59")
+    (pin "6")
+    (pin "60")
+    (pin "61")
+    (pin "62")
+    (pin "63")
+    (pin "64")
+    (pin "7")
+    (pin "8")
+    (pin "9")
+    (instances
+      (project "OrbitESC"
+        (path "/a13534e1-2c37-4692-a99c-4eada4007967/ed067bb8-caa7-448e-917b-cc2d33c8b4b7"
+          (reference "U3") (unit 1)
+        )
+      )
+    )
+  )
   (symbol (lib_id "power:GNDD") (at 134.62 156.845 270) (unit 1)
     (in_bom yes) (on_board yes) (dnp no)
@@
         )
       )
+    )
+  )
+  (symbol (lib_id "Connector:Micro_SD_Card") (at 240.665 232.41 0) (unit 1)
+    (in_bom yes) (on_board yes) (dnp no) (fields_autoplaced)
+    (property "Reference" "J13" (at 241.3 214.63 0)
+      (effects (font (size 1.27 1.27)))
+    )
+    (property "Value" "Micro_SD_Card" (at 241.3 217.17 0)
+      (effects (font (size 1.27 1.27)))
+    )
+    (property "Footprint" "" (at 269.875 224.79 0)
+      (effects (font (size 1.27 1.27)) hide)
+    )
+    (property "Datasheet" "http://katalog.we-online.de/em/datasheet/693072010801.pdf" (at 240.665 232.41 0)
+      (effects (font (size 1.27 1.27)) hide)
+    )
+    (pin "1")
+    (pin "2")
+    (pin "3")
+    (pin "4")
+    (pin "5")
+    (pin "6")
+    (pin "7")
+    (pin "8")
+    (pin "9")
+    (instances
+      (project "OrbitESC"
+        (path "/a13534e1-2c37-4692-a99c-4eada4007967/ed067bb8-caa7-448e-917b-cc2d33c8b4b7"
+          (reference "J13") (unit 1)
+        )
+      )

Commit message: Save some PCB work
Parts:
- removed C35, C55: 100nF, Capacitor_SMD:C_0402_1005Metric, symbol Device:C
- removed J11: RX, TestPoint:TestPoint_Pad_1.5x1.5mm, symbol Connector:Conn_01x01_Female
- removed J11: CANH, TestPoint:TestPoint_Pad_1.5x1.5mm, symbol Connector:Conn_01x01_Female
- removed J11: GND, TestPoint:TestPoint_Pad_1.5x1.5mm, symbol Connector:Conn_01x01_Female
- removed J11: TX, TestPoint:TestPoint_Pad_1.5x1.5mm, symbol Connector:Conn_01x01_Female
- removed J11: CANL, TestPoint:TestPoint_Pad_1.5x1.5mm, symbol Connector:Conn_01x01_Female
- removed R3, R70: 10k, Resistor_SMD:R_0402_1005Metric, symbol Device:R_US
- removed R62: 120, Resistor_SMD:R_0402_1005Metric, symbol Device:R_US
- removed TP10: NOR_SCK, TestPoint:TestPoint_Pad_D1.0mm, symbol Connector:TestPoint_Small
- removed TP13: NOR_MISO, TestPoint:TestPoint_Pad_D1.0mm, symbol Connector:TestPoint_Small
- removed TP9: NOR_MOSI, TestPoint:TestPoint_Pad_D1.0mm, symbol Connector:TestPoint_Small
- removed U11: STM32L432KCU6, Package_DFN_QFN:QFN-32-1EP_5x5mm_P0.5mm_EP3.45x3.45mm, symbol MCU_ST_STM32L4:STM32L432KBUx
- added C13, C32, C4, C7: 100nF, Capacitor_SMD:C_0402_1005Metric, symbol Device:C
- added D15, D18: Green LED, Diode_SMD:D_0603_1608Metric, symbol Device:LED
- added D20: Red LED, Diode_SMD:D_0603_1608Metric, symbol Device:LED
- added D5 (x2): Yellow LED, Diode_SMD:D_0603_1608Metric, symbol Device:LED
- added J1: USB_C_Receptacle_USB2.0, Connector_USB:USB_C_Receptacle_GCT_USB4085, symbol Connector:USB_C_Receptacle_USB2.0
- added J11: GND, TestPoint:TestPoint_Pad_1.5x1.5mm, symbol Connector:Conn_01x01_Female
- added J11: CANH, TestPoint:TestPoint_Pad_1.5x1.5mm, symbol Connector:Conn_01x01_Female
- added J11: CANL, TestPoint:TestPoint_Pad_1.5x1.5mm, symbol Connector:Conn_01x01_Female
- added R13, R9: 5.1k, Resistor_SMD:R_0402_1005Metric, symbol Device:R_US
- added R15: 120, Resistor_SMD:R_0402_1005Metric, symbol Device:R_US
- added R23, R53, R55, R86, R89: 10k, Resistor_SMD:R_0402_1005Metric, symbol Device:R_US
- added R56: 82k, symbol Device:R_US
- added R57: 33k, symbol Device:R_US
- added R7 (x2): 470, Resistor_SMD:R_0402_1005Metric, symbol Device:R_US
- added R91: 1.5k, Resistor_SMD:R_0402_1005Metric, symbol Device:R_US
- added SW2: DFU, Button_Switch_SMD:SW_SPST_PTS810, symbol Switch:SW_Push
- added TP3: NOR_MOSI, TestPoint:TestPoint_Pad_D1.0mm, symbol Connector:TestPoint_Small
- added TP4: NOR_SCK, TestPoint:TestPoint_Pad_D1.0mm, symbol Connector:TestPoint_Small
- added TP6: NOR_MISO, TestPoint:TestPoint_Pad_D1.0mm, symbol Connector:TestPoint_Small
- R42: value 120 -> 10k; LCSC C25079 -> C25744
- TP2: value NOR_MISO -> NOR_nCS
- TP5: value NOR_nCS -> NOR_MISO
Connections:
- net +3.3V: now also J10.1 (Pin_1), U3.19 (VDD), U3.32 (VDD), U3.48 (VDD), U3.64 (VDD), C4.2, C7.2, R23.2, R55.2, SW2.1; no longer R42.2
- net +3.3VADC: now also U3.13 (VDDA)
- net CAN1_RXD: now also U3.44 (PA11)
- net CAN1_TXD: now also U3.45 (PA12)
- net GATE_DRIVE_AH: now also U3.41 (PA8)
- net GATE_DRIVE_AL: now also U3.23 (PA7)
- net GATE_DRIVE_BH: now also U3.42 (PA9)
- net GATE_DRIVE_BL: now also U3.26 (PB0)
- net GATE_DRIVE_CH: now also U3.43 (PA10)
- net GATE_DRIVE_CL: now also U3.27 (PB1)
- net GND: now also R42.1, TP5.1, U3.12 (VSSA), U3.18 (VSS), U3.31 (VSS), U3.47 (VSS), U3.63 (VSS), C13.2, C32.1, C4.1, C7.1, D15.1 (K), D18.1 (K), D20.1 (K), D5.1 (K), D5.1 (K), J1.A1 (GND), J1.A12 (GND), J1.B1 (GND), J1.B12 (GND), J1.S1 (SHIELD), J11.1 (Pin_1), R13.2, R53.1, R56.2, R9.1; no longer TP2.1
- net MOTOR_IA: now also U3.14 (PA0)
- net MOTOR_IB: now also U3.15 (PA1)
- net MOTOR_VA: now also U3.17 (PA3)
- net MOTOR_VB: now also U3.20 (PA4)
- net MOTOR_VC: now also U3.21 (PA5)
- net NOR_MISO: now also U3.56 (PB4), TP6.1
- net NOR_MOSI: now also U3.57 (PB5), TP3.1
- net NOR_SCK: now also U3.55 (PB3), TP4.1
- net NOR_nCS: now also TP2.1, U3.50 (PA15), R55.1; no longer TP5.1
- net SERIAL1_IN: now also U3.38 (PC7)
- net SERIAL1_OUT: now also U3.37 (PC6)
- net SWCLK: now also U3.49 (PA14)
- net SWDIO: now also U3.46 (PA13)
- net VS: now also U3.8 (PC0); no longer C13.1, R23.1, R24.1
- net VTEMP: now also U3.9 (PC1)
- net nRESET: now also U3.7 (NRST)
- net at U1.7 (CANH): now also J11.1 (Pin_1), R15.2
- net at U1.6 (CANL): now also J11.1 (Pin_1), R15.1
- net MOTOR_IC: now reaches U3.16 (PA2)
- net USBActiveLED: now reaches U3.2 (PC13)
- net USBActiveLED: now also R7.1
- net at U3.34 (PB13): now also R56.1, R57.2
- net USB_D-: now reaches U3.35 (PB14)
- net USB_D-: now also J1.A7 (D-), J1.B7 (D-)
- net USB_D+: now reaches U3.36 (PB15)
- net USB_D+: now also J1.A6 (D+), J1.B6 (D+)
- net SDIO_D0: now reaches U3.39 (PC8)
- net SDIO_D0: now also J13.7 (DAT0)
- net SDIO_D1: now reaches U3.40 (PC9)
- net SDIO_D1: now also J13.8 (DAT1)
- net SDIO_D2: now reaches U3.51 (PC10)
- net SDIO_D2: now also J13.1 (DAT2)
- net SDIO_D3: now reaches U3.52 (PC11)
- net SDIO_D3: now also J13.2 (DAT3/CD)
- net SDIO_CLK: now reaches U3.53 (PC12)
- net SDIO_CLK: now also J13.5 (CLK)
- net SDIO_CMD: now reaches U3.54 (PD2)
- net SDIO_CMD: now also J13.3 (CMD)
- net FaultLED: now reaches U3.58 (PB6)
- net FaultLED: now also R91.1
- net ArmedLED: now reaches U3.59 (PB7)
- net ArmedLED: now also R89.1
- net nDFU_BOOT: now reaches U3.60 (BOOT0)
- net nDFU_BOOT: now also R42.2, C32.2, SW2.2
- net HeartbeatLED: now reaches U3.61 (PB8)
- net HeartbeatLED: now also R86.1
- net CANActiveLED: now reaches U3.62 (PB9)
- net CANActiveLED: now also R7.1
- new net: D18.2 (A), R89.2
- new net: D15.2 (A), R86.2
- new net: J1.B5 (CC2), R13.1
- new net: D20.2 (A), R91.2
- new net: D5.2 (A), R7.2 (x2)
- new net: J1.A5 (CC1), R9.2
- new net VBUS: J1.A4 (VBUS), J1.A9 (VBUS), J1.B4 (VBUS), J1.B9 (VBUS), R57.1
- new net VMCU: C13.1, R23.1, R53.2
- new net VSUPPLY: C13.1, R23.1, R24.1
- no-connect marks 4 -> 14
Other:
- removed sheet Status LEDs
- removed sheet USB2Serial
- note added: "Need: 1. Oscillator 2. ADC assignments 3. Validate USB connections 4. Validate SDIO connections 5. Validate Power supply"
- note removed: "Keep both SPI and SD card for now"
- note removed: "Power Stage Temperature"
- note removed: "Supply Voltage Sense"
- moved on the sheet: C1, C13, C29, J10, J13, R1, R20, R23, R24, SW1, TH1, U3

Commit message: PCB work over lunch
Parts:
- added C29: 4.7uF, Capacitor_SMD:C_0402_1005Metric, symbol Device:C
- added C35, C36, C48, C49: 100nF, Capacitor_SMD:C_0402_1005Metric, symbol Device:C
- added X1: ASE-24MHz, Oscillator:Oscillator_SMD_Abracon_ASE-4Pin_3.2x2.5mm, symbol Oscillator:ASE-xxxMHz
- renumbered D5 to D4, D15 to D5, D18 to D6, D20 to D7, D5 to D9, R86 to R19, R89 to R29, R91 to R52, R7 to R58
Connections:
- net VS is gone; now on net VSUPPLY: U3.8 (PC0)
- net +3.3V: now also C35.2, C48.2, C49.2, X1.4 (Vdd)
- net GND: now also C29.1, C35.1, C36.2, C48.1, C49.1, X1.2 (GND)
- net VMCU: now also U3.10 (PC2)
- net VISENSE_REF: now reaches U3.11 (PC3)
- net at U3.30 (VCAP_1): now also C29.2, C36.1
- net at U3.5 (PH0): now also X1.3 (OUT)
- no-connect marks 14 -> 17
Other:
- note removed: "Join at single point"
