File: hw/pcb/OrbitESC_V3/microcontroller.kicad_sch (KiCad schematic)
At the start: 58 parts, among them J1 USB_C_Receptacle_USB2.0, J11 CANH, J11 CANL, J11 GND, J11 RX, J11 TX, J8 Micro_SD_Card_Det2, SW1 Reset, SW2 DFU, U1 TLE9250X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

Commit message: Merge branch 'feature/pcb_v3_bringup/r0'
Other:
- note added: "Need to add an inline power switch to control initialization behavior."
- note added: "Packaging is wrong for this chip? Atleast compared to what I ordered."
- note added: "Possibly add 10k pull ups on these lines. I can't seem to run at a bus speed greater than 4MHz. Also need to length match all the lines."
- note added: "Pretty sure this resistor is preventing DFU from working b/c the pullup never goes high with STM32 bootloader code. I could try using a PNP transitor to invert the logic? I'm not sure I want the extra parts though. Update 10/28/2023: Turns out that this resistor is already embedded on the F446RE and including it under GPIO control is really messing with my software. Remove it."
- note added: "VBus sensing can be removed. When the F4 configures PA9 as an alternate function, it breaks sensing. Solution is to disable/override sensing in software and force device mode."
- note removed: "Packaging is wrong for this chip?"
- note removed: "Pretty sure this resistor is preventing DFU from working b/c the pullup never goes high with STM32 bootloader code."
Changed lines of the file:
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@@
     (stroke (width 0) (type default))
   )
-  (text "Packaging is wrong for this chip?" (at 274.955 131.445 0)
+  (text "Need to add an inline power switch to control initialization behavior."
+    (at 247.65 171.45 0)
     (effects (font (size 1.27 1.27)) (justify left bottom))
   )
-  (text "Pretty sure this resistor is preventing DFU from working\nb/c the pullup never goes high with STM32 bootloader code."
-    (at 273.05 243.84 0)
+  (text "Packaging is wrong for this chip? Atleast compared to what I ordered."
+    (at 252.095 144.145 0)
     (effects (font (size 1.27 1.27)) (justify left bottom))
   )
+  (text "Possibly add 10k pull ups on these lines. I can't seem\nto run at a bus speed greater than 4MHz. Also need to length\nmatch all the lines."
+    (at 233.045 182.88 0)
+    (effects (font (size 1.27 1.27)) (justify left bottom))
+  )
+  (text "Pretty sure this resistor is preventing DFU from working\nb/c the pullup never goes high with STM32 bootloader code.\nI could try using a PNP transitor to invert the logic? I'm\nnot sure I want the extra parts though.\n\nUpdate 10/28/2023: Turns out that this resistor is already\nembedded on the F446RE and including it under GPIO control\nis really messing with my software. Remove it."
+    (at 243.205 254 0)
+    (effects (font (size 1.27 1.27)) (justify left bottom))
+  )
+  (text "VBus sensing can be removed. When the F4 configures PA9 as\nan alternate function, it breaks sensing. Solution is to \ndisable/override sensing in software and force device mode."
+    (at 240.665 228.6 0)
+    (effects (font (size 1.27 1.27)) (justify left bottom))
+  )
