File: hw/pcb/OrbitESC_V3/OrbitESC.kicad_pcb (KiCad board)
At the start: 8 copper layers, 45.2 x 29.7 mm, 159 parts, among them J1 USB_C_Receptacle_USB2.0, J11 VDC, J12 GND, J13 RX, J2 CANH, J3 TermA, J4 TermB, J5 TermC, J6 GND, J7 CANL, J8 Micro_SD_Card_Det2, J9 TX, Q1 MCAC100N08YA-TP, Q2 MCAC100N08YA-TP, Q3 MCAC100N08YA-TP, Q4 MCAC100N08YA-TP, Q5 MCAC100N08YA-TP, Q6 MCAC100N08YA-TP, Q7 2N7002, SW1 Reset, SW2 DFU, U1 TLE9250X, U13 TLV9051IDBVR, U14 TLV9051IDBVR, U2 AT25SF128A-SHB-T, U3 STM32F446RETx, U4 TLV9051IDBVR, U5 DRV8300DRGER, U6 TLV9051IDBVR, U7 AP62200Z6-7, U8 AP2171W, U9 AP2120, X1 ASE-24MHz

Commit message: Finalize PCB. Ordered it.
Parts:
- added TP1: CH, TestPoint:TestPoint_Pad_D1.0mm, B.Cu at (189.6, 63.1)
- added TP2: CH, TestPoint:TestPoint_Pad_D1.0mm, B.Cu at (191.6, 63.1)
Connections:
- U3 pad 24: unconnected-(U3-PC4-Pad24) -> Net-(U3-PC4)
- U3 pad 25: unconnected-(U3-PC5-Pad25) -> Net-(U3-PC5)
Routing:
- net Net-(U3-PC5): track 0.00 -> 27.9 mm, vias 0 -> 2
- net Net-(U3-PC4): track 0.00 -> 20.1 mm, vias 0 -> 2
