File: hw/pcb/OrbitESC_V3/OrbitESC.kicad_sch (KiCad schematic)
At the start: 0 parts

Commit message: Save some PCB work
Other:
- sheet MCU ports: added MOTOR_IC; removed none
Changed lines of the file:
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@@
+      (effects (font (size 1.27 1.27)) (justify right))
+    )
+    (pin "MOTOR_IC" input (at 158.115 95.25 0)
       (effects (font (size 1.27 1.27)) (justify right))
     )

Commit message: PCB work over lunch
Other:
- sheet MCU ports: added VISENSE_REF; removed none
- sheet Outputs and Shunts ports: added C_ISENSE_N, C_ISENSE_P; removed none
- sheet Power Stage ports: added C_ISENSE_N, C_ISENSE_P, IC, ISenseVRef; removed none
Changed lines of the file:
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@@
+    (stroke (width 0) (type default))
+  )
+  (wire (pts (xy 158.115 87.63) (xy 163.83 87.63))
+    (stroke (width 0) (type default))
+  )
+  (wire (pts (xy 158.115 95.25) (xy 163.83 95.25))
+    (stroke (width 0) (type default))
+  )
+  (wire (pts (xy 199.39 110.49) (xy 202.565 110.49))
     (stroke (width 0) (type default))
   )
@@
   )
   (wire (pts (xy 158.115 97.79) (xy 163.83 97.79))
+    (stroke (width 0) (type default))
+  )
+  (wire (pts (xy 199.39 107.95) (xy 202.565 107.95))
     (stroke (width 0) (type default))
   )
@@
       (effects (font (size 1.27 1.27)) (justify left))
     )
+    (pin "C_ISENSE_P" output (at 202.565 107.95 180)
+      (effects (font (size 1.27 1.27)) (justify left))
+    )
+    (pin "C_ISENSE_N" output (at 202.565 110.49 180)
+      (effects (font (size 1.27 1.27)) (justify left))
+    )
     (instances
       (project "OrbitESC"
@@
       (effects (font (size 1.27 1.27)) (justify left))
     )
+    (pin "ISenseVRef" output (at 163.83 87.63 180)
+      (effects (font (size 1.27 1.27)) (justify left))
+    )
+    (pin "IC" output (at 163.83 95.25 180)
+      (effects (font (size 1.27 1.27)) (justify left))
+    )
+    (pin "C_ISENSE_P" input (at 199.39 107.95 0)
+      (effects (font (size 1.27 1.27)) (justify right))
+    )
+    (pin "C_ISENSE_N" input (at 199.39 110.49 0)
+      (effects (font (size 1.27 1.27)) (justify right))
+    )
     (instances
       (project "OrbitESC"
@@
       (effects (font (size 1.27 1.27)) (justify right))
     )
+    (pin "VISENSE_REF" input (at 158.115 87.63 0)
+      (effects (font (size 1.27 1.27)) (justify right))
+    )
