File: hw/pcb/OrbitESC_V3/output_stage.kicad_sch (KiCad schematic)
At the start: 19 parts, among them J3 TermA, J4 TermB, J5 TermC, Q1 MCAC100N08YA-TP, Q2 MCAC100N08YA-TP, Q3 MCAC100N08YA-TP, Q4 MCAC100N08YA-TP, Q5 MCAC100N08YA-TP, Q6 MCAC100N08YA-TP

Commit message: PCB work over lunch
Parts:
- added C45: 1nF, Capacitor_SMD:C_0402_1005Metric, symbol Device:C
- added R63: 0.01, Resistor_SMD:R_2512_6332Metric, symbol Device:R_US
Connections:
- net GND: now also C45.2, R63.2; no longer Q6.3 (S)
- new net C_ISENSE_P: C45.1, Q6.3 (S), R63.1
Changed lines of the file:
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@@
   (junction (at 80.01 120.65) (diameter 0) (color 0 0 0 0)
   )
+  (junction (at 255.27 120.65) (diameter 0) (color 0 0 0 0)
+  )
   (junction (at 80.01 83.82) (diameter 0) (color 0 0 0 0)
   )
@@
   (junction (at 157.48 120.65) (diameter 0) (color 0 0 0 0)
   )
+  (junction (at 255.27 107.95) (diameter 0) (color 0 0 0 0)
+  )
   (junction (at 69.85 120.65) (diameter 0) (color 0 0 0 0)
   )
+  (junction (at 245.11 107.95) (diameter 0) (color 0 0 0 0)
+  )
   (junction (at 167.64 107.95) (diameter 0) (color 0 0 0 0)
   )
+  (junction (at 245.11 120.65) (diameter 0) (color 0 0 0 0)
+  )
   (junction (at 167.64 120.65) (diameter 0) (color 0 0 0 0)
   )
@@
     (stroke (width 0) (type default))
   )
+  (wire (pts (xy 255.27 107.95) (xy 255.27 102.87))
+    (stroke (width 0) (type default))
+  )
   (wire (pts (xy 212.09 71.12) (xy 234.95 71.12))
     (stroke (width 0) (type default))
@@
     (stroke (width 0) (type default))
   )
+  (wire (pts (xy 212.09 107.95) (xy 245.11 107.95))
+    (stroke (width 0) (type default))
+  )
   (wire (pts (xy 157.48 118.11) (xy 157.48 120.65))
     (stroke (width 0) (type default))
@@
     (stroke (width 0) (type default))
   )
+  (wire (pts (xy 245.11 107.95) (xy 245.11 110.49))
+    (stroke (width 0) (type default))
+  )
   (wire (pts (xy 80.01 107.95) (xy 80.01 110.49))
     (stroke (width 0) (type default))
@@
     (stroke (width 0) (type default))
   )
+  (wire (pts (xy 245.11 107.95) (xy 255.27 107.95))
+    (stroke (width 0) (type default))
+  )
+  (wire (pts (xy 212.09 120.65) (xy 245.11 120.65))
+    (stroke (width 0) (type default))
+  )
   (wire (pts (xy 124.46 107.95) (xy 157.48 107.95))
     (stroke (width 0) (type default))
@@
     (stroke (width 0) (type default))
   )
+  (wire (pts (xy 245.11 120.65) (xy 255.27 120.65))
+    (stroke (width 0) (type default))
+  )
   (wire (pts (xy 36.83 71.12) (xy 59.69 71.12))
     (stroke (width 0) (type default))
   )
+  (wire (pts (xy 255.27 118.11) (xy 255.27 120.65))
+    (stroke (width 0) (type default))
+  )
   (wire (pts (xy 69.85 107.95) (xy 80.01 107.95))
     (stroke (width 0) (type default))
@@
     (stroke (width 0) (type default))
   )
+  (wire (pts (xy 255.27 107.95) (xy 255.27 110.49))
+    (stroke (width 0) (type default))
+  )
   (wire (pts (xy 80.01 59.69) (xy 80.01 66.04))
     (stroke (width 0) (type default))
@@
     (stroke (width 0) (type default))
   )
+  (wire (pts (xy 245.11 118.11) (xy 245.11 120.65))
+    (stroke (width 0) (type default))
+  )
   (hierarchical_label "GDH_C" (shape input) (at 212.09 71.12 180) (fields_autoplaced)
     (effects (font (size 1.27 1.27)) (justify right))
@@
     (effects (font (size 1.27 1.27)) (justify right))
   )
+  (hierarchical_label "C_ISENSE_N" (shape output) (at 212.09 120.65 180) (fields_autoplaced)
+    (effects (font (size 1.27 1.27)) (justify right))
+  )
   (hierarchical_label "GDL_C" (shape input) (at 212.09 97.79 180) (fields_autoplaced)
     (effects (font (size 1.27 1.27)) (justify right))
   )
+  (hierarchical_label "C_ISENSE_P" (shape output) (at 212.09 107.95 180) (fields_autoplaced)
+    (effects (font (size 1.27 1.27)) (justify right))
+  )
   (hierarchical_label "SH_C" (shape output) (at 242.57 83.82 180) (fields_autoplaced)
     (effects (font (size 1.27 1.27)) (justify right))
@@
     (effects (font (size 1.27 1.27)) (justify right))
   )
+  (symbol (lib_id "Device:C") (at 245.11 114.3 0) (unit 1)
+    (in_bom yes) (on_board yes) (dnp no) (fields_autoplaced)
+    (property "Reference" "C45" (at 248.92 113.0299 0)
+      (effects (font (size 1.27 1.27)) (justify left))
+    )
+    (property "Value" "1nF" (at 248.92 115.5699 0)
+      (effects (font (size 1.27 1.27)) (justify left))
+    )
+    (property "Footprint" "Capacitor_SMD:C_0402_1005Metric" (at 246.0752 118.11 0)
+      (effects (font (size 1.27 1.27)) hide)
+    )
+    (property "Datasheet" "~" (at 245.11 114.3 0)
+      (effects (font (size 1.27 1.27)) hide)
+    )
+    (property "JLCPCB" "" (at 245.11 114.3 0)
+      (effects (font (size 1.27 1.27)) hide)
+    )
+    (property "LCSC" "C1523" (at 245.11 114.3 0)
+      (effects (font (size 1.27 1.27)) hide)
+    )
+    (pin "1")
+    (pin "2")
+    (instances
+      (project "OrbitESC"
+        (path "/a13534e1-2c37-4692-a99c-4eada4007967/01eceaba-0372-470e-b19c-b8e61f77bd53"
+          (reference "C45") (unit 1)
+        )
+      )
+    )
+  )
   (symbol (lib_id "Project Mosfets:MCAC80N10Y") (at 165.1 97.79 0) (unit 1)
     (in_bom yes) (on_board yes) (dnp no) (fields_autoplaced)
@@
     )
   )
-  (symbol (lib_id "power:GND") (at 255.27 102.87 0) (unit 1)
-    (in_bom yes) (on_board yes) (dnp no) (fields_autoplaced)
-    (property "Reference" "#PWR011" (at 255.27 109.22 0)
-      (effects (font (size 1.27 1.27)) hide)
-    )
-    (property "Value" "GND" (at 255.27 107.95 0)
-      (effects (font (size 1.27 1.27)))
-    )
-    (property "Footprint" "" (at 255.27 102.87 0)
-      (effects (font (size 1.27 1.27)) hide)
-    )
-    (property "Datasheet" "" (at 255.27 102.87 0)
-      (effects (font (size 1.27 1.27)) hide)
-    )
-    (pin "1")
-    (instances
-      (project "OrbitESC"
-        (path "/a13534e1-2c37-4692-a99c-4eada4007967/01eceaba-0372-470e-b19c-b8e61f77bd53"
-          (reference "#PWR011") (unit 1)
+  (symbol (lib_id "power:GND") (at 255.27 120.65 0) (unit 1)
+    (in_bom yes) (on_board yes) (dnp no) (fields_autoplaced)
+    (property "Reference" "#PWR097" (at 255.27 127 0)
+      (effects (font (size 1.27 1.27)) hide)
+    )
+    (property "Value" "GND" (at 255.27 125.73 0)
+      (effects (font (size 1.27 1.27)))
+    )
+    (property "Footprint" "" (at 255.27 120.65 0)
+      (effects (font (size 1.27 1.27)) hide)
+    )
+    (property "Datasheet" "" (at 255.27 120.65 0)
+      (effects (font (size 1.27 1.27)) hide)
+    )
+    (pin "1")
+    (instances
+      (project "OrbitESC"
+        (path "/a13534e1-2c37-4692-a99c-4eada4007967/01eceaba-0372-470e-b19c-b8e61f77bd53"
+          (reference "#PWR097") (unit 1)
         )
       )
@@
         )
       )
+    )
+  )
+  (symbol (lib_id "Device:R_US") (at 255.27 114.3 0) (unit 1)
+    (in_bom yes) (on_board yes) (dnp no) (fields_autoplaced)
+    (property "Reference" "R63" (at 257.81 113.0299 0)
+      (effects (font (size 1.27 1.27)) (justify left))
+    )
+    (property "Value" "0.01" (at 257.81 115.5699 0)
+      (effects (font (size 1.27 1.27)) (justify left))
+    )
+    (property "Footprint" "Resistor_SMD:R_2512_6332Metric" (at 256.286 114.554 90)
+      (effects (font (size 1.27 1.27)) hide)
+    )
+    (property "Datasheet" "~" (at 255.27 114.3 0)
+      (effects (font (size 1.27 1.27)) hide)
+    )
+    (property "DigiKey" "CRA2512-FZ-R010ELFCT-ND" (at 255.27 114.3 0)
+      (effects (font (size 1.27 1.27)) hide)
+    )
+    (pin "1")
+    (pin "2")
+    (instances
+      (project "OrbitESC"
+        (path "/a13534e1-2c37-4692-a99c-4eada4007967/01eceaba-0372-470e-b19c-b8e61f77bd53"
+          (reference "R63") (unit 1)
+        )
+      )
