File: hw/pcb/OrbitESC_V3/power_stage.kicad_sch (KiCad schematic)
At the start: 53 parts, among them U13 TLV9051IDBVR, U14 TLV9051IDBVR, U4 TLV9051IDBVR, U5 DRV8300DRGER

Commit message: PCB work over lunch
Parts:
- added C38: 4.7nF, Capacitor_SMD:C_0402_1005Metric, symbol Device:C
- added C40: 100nF, Capacitor_SMD:C_0402_1005Metric, symbol Device:C
- added R3, R59, R62: 10k, Resistor_SMD:R_0402_1005Metric, symbol Device:R_US
- added R60, R61: 1k, Resistor_SMD:R_0402_1005Metric, symbol Device:R_US
- added TP9: AH, TestPoint:TestPoint_Pad_D1.0mm, symbol Connector:TestPoint_Small
- added U6: TLV9051IDBVR, Package_TO_SOT_SMD:SOT-23-5, symbol Amplifier_Operational:TLV9001IDCK
- renumbered C32 to C13, C32 to C22, C32 to C23, C32 to C8, C32 to C9
Connections:
- net +3.3VADC: now also C40.1, U6.5 (V+)
- net GND: now also C38.1, C40.2, U6.2 (V-)
- net ISenseVRef: now also R62.2
- new net: R3.2, R59.1, U6.1
- new net: R61.2, R62.1, U6.3 (+)
- new net: R59.2, R60.2, U6.4 (-)
- new net C_ISENSE_N: R61.1
- new net C_ISENSE_P: R60.1
- new net IC: C38.2, R3.1, TP9.1
Other:
- moved on the sheet: C12, C13, C14, C16, C22, C23, C30, C42, C43, C44, C8, C9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

Commit message: Semi-final schematic for F4 variant
Parts:
- removed C23, C38, C8: 4.7nF, Capacitor_SMD:C_0402_1005Metric, symbol Device:C
- removed R18, R25, R26, R27, R28, R3: 10k, Resistor_SMD:R_0402_1005Metric, symbol Device:R_US
Connections:
- net IA: now also R34.1, U14.1
- net IB: now also R31.1, U13.1
- net IC: now also R59.1, U6.1
- net SHA: now also C9.2, R45.2
- net SHB: now also C13.2, R49.2
- net SHC: now also C22.2, R51.2

Commit message: Finish initial draft of V3 pcb
Parts:
- removed TP1: BL, TestPoint:TestPoint_Pad_D1.0mm, symbol Connector:TestPoint_Small
- removed TP7, TP8, TP9: AH, TestPoint:TestPoint_Pad_D1.0mm, symbol Connector:TestPoint_Small
Other:
- note removed: "3.3KHz LPF"

Commit message: PCB cleanup. BOM checks.
Parts:
- R45, R49, R51: value 18k -> 39k; LCSC C25762 -> C25783
- R46, R48, R50: value 1k -> 5.1k; LCSC C11702 -> C25905
- TP14, TP15, TP16, TP17, TP18, TP19: DigiKey (none) -> N/A
Changed lines of the file:
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@@
       (effects (font (size 1.27 1.27)))
     )
-    (property "Value" "18k" (at 233.045 72.39 90)
+    (property "Value" "39k" (at 233.045 72.39 90)
       (effects (font (size 1.27 1.27)))
     )
@@
       (effects (font (size 1.27 1.27)) hide)
     )
-    (property "LCSC" "C25762" (at 233.045 76.2 0)
+    (property "LCSC" "C25783" (at 233.045 76.2 0)
       (effects (font (size 1.27 1.27)) hide)
     )
@@
       (effects (font (size 1.27 1.27)) (justify right))
     )
-    (property "Value" "1k" (at 228.6 60.325 0)
+    (property "Value" "5.1k" (at 228.6 60.325 0)
       (effects (font (size 1.27 1.27)) (justify right))
     )
@@
       (effects (font (size 1.27 1.27)) hide)
     )
-    (property "LCSC" "C11702" (at 226.695 58.42 0)
+    (property "LCSC" "C25905" (at 226.695 58.42 0)
       (effects (font (size 1.27 1.27)) hide)
     )
@@
       (effects (font (size 1.27 1.27)) hide)
     )
+    (property "DigiKey" "N/A" (at 114.3 32.385 0)
+      (effects (font (size 1.27 1.27)) hide)
+    )
     (pin "1")
     (instances
@@
       (effects (font (size 1.27 1.27)))
     )
-    (property "Value" "18k" (at 233.045 26.67 90)
+    (property "Value" "39k" (at 233.045 26.67 90)
       (effects (font (size 1.27 1.27)))
     )
@@
       (effects (font (size 1.27 1.27)) hide)
     )
-    (property "LCSC" "C25762" (at 233.045 30.48 0)
+    (property "LCSC" "C25783" (at 233.045 30.48 0)
       (effects (font (size 1.27 1.27)) hide)
     )
@@
       (effects (font (size 1.27 1.27)) hide)
     )
+    (property "DigiKey" "N/A" (at 114.3 42.545 0)
+      (effects (font (size 1.27 1.27)) hide)
+    )
     (pin "1")
     (instances
@@
     )
     (property "Datasheet" "~" (at 119.38 40.005 0)
+      (effects (font (size 1.27 1.27)) hide)
+    )
+    (property "DigiKey" "N/A" (at 114.3 40.005 0)
       (effects (font (size 1.27 1.27)) hide)
     )
@@
       (effects (font (size 1.27 1.27)) hide)
     )
+    (property "DigiKey" "N/A" (at 114.3 47.625 0)
+      (effects (font (size 1.27 1.27)) hide)
+    )
     (pin "1")
     (instances
@@
       (effects (font (size 1.27 1.27)) (justify right))
     )
-    (property "Value" "1k" (at 228.6 37.465 0)
+    (property "Value" "5.1k" (at 228.6 37.465 0)
       (effects (font (size 1.27 1.27)) (justify right))
     )
@@
       (effects (font (size 1.27 1.27)) hide)
     )
-    (property "LCSC" "C11702" (at 226.695 35.56 0)
+    (property "LCSC" "C25905" (at 226.695 35.56 0)
       (effects (font (size 1.27 1.27)) hide)
     )
@@
       (effects (font (size 1.27 1.27)))
     )
-    (property "Value" "18k" (at 233.045 49.53 90)
+    (property "Value" "39k" (at 233.045 49.53 90)
       (effects (font (size 1.27 1.27)))
     )
@@
       (effects (font (size 1.27 1.27)) hide)
     )
-    (property "LCSC" "C25762" (at 233.045 53.34 0)
+    (property "LCSC" "C25783" (at 233.045 53.34 0)
       (effects (font (size 1.27 1.27)) hide)
     )
@@
       (effects (font (size 1.27 1.27)) hide)
     )
+    (property "DigiKey" "N/A" (at 114.3 34.925 0)
+      (effects (font (size 1.27 1.27)) hide)
+    )
     (pin "1")
     (instances
@@
       (effects (font (size 1.27 1.27)) hide)
     )
+    (property "DigiKey" "N/A" (at 114.3 50.165 0)
+      (effects (font (size 1.27 1.27)) hide)
+    )
     (pin "1")
     (instances
@@
       (effects (font (size 1.27 1.27)) (justify right))
     )
-    (property "Value" "1k" (at 228.6 83.185 0)
+    (property "Value" "5.1k" (at 228.6 83.185 0)
       (effects (font (size 1.27 1.27)) (justify right))
     )
@@
       (effects (font (size 1.27 1.27)) hide)
     )
-    (property "LCSC" "C11702" (at 226.695 81.28 0)
-      (effects (font (size 1.27 1.27)) hide)
-    )
+    (property "LCSC" "C25905" (at 226.695 81.28 0)
+      (effects (font (size 1.27 1.27)) hide)
+    )
