File: hw/pcb/OrbitESC_V3/power_supply.kicad_sch (KiCad schematic)
At the start: 33 parts, among them J11 VDC, J12 GND, Q7 2N7002, U7 AP62200Z6-7, U8 AP2171W, U9 AP2120

Commit message: PCB cleanup. BOM checks.
Parts:
- R40: DigiKey RMCF0402FT57K6CT-ND -> (none)
Changed lines of the file:
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@@
       (effects (font (size 1.27 1.27)) hide)
     )
-    (property "DigiKey" "RMCF0402FT57K6CT-ND" (at 176.53 38.1 0)
+    (property "DigiKey" "" (at 176.53 38.1 0)
       (effects (font (size 1.27 1.27)) hide)
     )

Commit message: Update schematic with a few discoveries from board bringup
Other:
- note added: "1k resistor here prevents boot up. Remove it."
Changed lines of the file:
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@@
+    (effects (font (size 1.27 1.27)) (justify left bottom))
+  )
+  (text "1k resistor here prevents boot up. Remove it." (at 165.1 114.3 0)
     (effects (font (size 1.27 1.27)) (justify left bottom))
   )
